Commit message: correct orientation on robot_test meshs files

File: data/urdf/robot_test/robot_test_lleg_rom.urdf (robot description, URDF)
Before this commit: robot robot_lleg_rom, 1 links, 0 joints
Links:
- link base_link: geometry collision mesh filename=package://hpp-rbprm-corba/meshes/robot_test/Lleg_rom.stl; visual mesh filename=package://hpp-rbprm-corba/meshes/robot_test/Lleg_rom.stl

File: data/urdf/robot_test/robot_test_rleg_rom.urdf (robot description, URDF)
Before this commit: robot robot_rleg_rom, 1 links, 0 joints
Links:
- link base_link: geometry collision mesh filename=package://hpp-rbprm-corba/meshes/robot_test/Rleg_rom.stl; visual mesh filename=package://hpp-rbprm-corba/meshes/robot_test/Rleg_rom.stl
