Commit message: add mass info in urdf file for robot_test

File: data/urdf/robot_test/robot_test_trunk.urdf (robot description, URDF)
Before this commit: robot robot_trunk, 1 links, 0 joints
Links:
- link base_link: mass None -> 50

Commit message: minor change in script

File: data/urdf/robot_test/robot_test_trunk.urdf (robot description, URDF)
Before this commit: robot robot_trunk, 1 links, 0 joints
Links:
- link base_link: mass 50 -> 10
