Commit message: correct urdf files for ground_jump_easy

File: data/urdf/ground_jump_easy.urdf (robot description, URDF)
Before this commit: robot ground_jump_easy, 1 links, 0 joints
Links:
- removed link base_link
- added link ground
- added link groundGoal; collision mesh filename=package://hpp-rbprm-corba/meshes/ground_jump_easyGoal.stl; visual mesh filename=package://hpp-rbprm-corba/meshes/ground_jump_easyGoal.stl
- added link groundStart; collision mesh filename=package://hpp-rbprm-corba/meshes/ground_jump_easyStart.stl; visual mesh filename=package://hpp-rbprm-corba/meshes/ground_jump_easyStart.stl
Joints:
- added joint ground_goal_joint: type fixed, parent ground, child groundGoal, origin xyz=0 0 0 rpy=0 0 0
- added joint ground_start_joint: type fixed, parent ground, child groundStart, origin xyz=0 0 0 rpy=0 0 0

File: data/urdf/robot_test/robot_test_lleg_rom.urdf (robot description, URDF)
Before this commit: robot robot_lleg_rom, 1 links, 0 joints
Links:
- removed link base_link
- added link llged_rom; collision mesh filename=package://hpp-rbprm-corba/meshes/robot_test/Lleg_rom.stl; visual mesh filename=package://hpp-rbprm-corba/meshes/robot_test/Lleg_rom.stl

File: data/urdf/robot_test/robot_test_rleg_rom.urdf (robot description, URDF)
Before this commit: robot robot_rleg_rom, 1 links, 0 joints
Links:
- removed link base_link
- added link rleg_rom; collision mesh filename=package://hpp-rbprm-corba/meshes/robot_test/Rleg_rom.stl; visual mesh filename=package://hpp-rbprm-corba/meshes/robot_test/Rleg_rom.stl

File: data/urdf/robot_test/robot_test_trunk.urdf (robot description, URDF)
Before this commit: robot robot_trunk, 1 links, 0 joints
Links:
- removed link base_link
- added link robot_trunk_root, mass 10; collision mesh filename=package://hpp-rbprm-corba/meshes/robot_test/robot_trunk.stl; visual mesh filename=package://hpp-rbprm-corba/meshes/robot_test/robot_trunk_vie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
