Commit message: update friction-less scenario and add ant script

File: data/urdf/cliff.urdf (robot description, URDF)
Before this commit: robot cubeWorld, 1 links, 0 joints
Links:
- link base_link: geometry collision mesh filename=package://hpp-rbprm-corba/meshes/cliff_panel.stl; visual mesh filename=package://hpp-rbprm-corba/meshes/cliff.stl
