Commit message: FIX trunk-ecsSize used in fullConfig TODO: propagate, add parkour-wall envir

File: data/urdf/parkour_walls.urdf (robot description, URDF)
Before this commit: robot obstacle, 1 links, 0 joints
Links:
- link base_link: geometry collision mesh filename=package://hpp-rbprm-corba/meshes/parkour_walls.stl; visual mesh filename=package://hpp-rbprm-corba/meshes/parkour_walls.stl
