Commit message: Add missing files for environment

File: data/urdf/cave.urdf (robot description, URDF)
Before this commit: robot obstacle, 1 links, 0 joints
Links:
- link base_link: geometry collision mesh filename=package://hpp-rbprm-corba/meshes/cave_simplified.stl; visual mesh filename=package://hpp-rbprm-corba/meshes/cave_simplified.stl

File: data/urdf/cubeWorld2.urdf (robot description, URDF)
Before this commit: robot cubeWorld, 1 links, 0 joints
Links:
- link base_link: geometry collision mesh filename=package://hpp-rbprm-corba/meshes/cubeWorld2.stl; visual mesh filename=package://hpp-rbprm-corba/meshes/cubeWorld2.stl

File: data/urdf/high_plateforms.urdf (robot description, URDF)
Before this commit: robot obstacle, 1 links, 0 joints
Links:
- link base_link: geometry collision mesh filename=package://hpp-rbprm-corba/meshes/high_plateforms.stl; visual mesh filename=package://hpp-rbprm-corba/meshes/high_plateforms.stl

File: data/urdf/parkour_walls.urdf (robot description, URDF)
Before this commit: robot obstacle, 1 links, 0 joints
Links:
- link base_link: geometry collision mesh filename=package://hpp-rbprm-corba/meshes/parkour_walls_reduced.stl; visual mesh filename=package://hpp-rbprm-corba/meshes/parkour_walls_reduced.stl
