Commit message: Modify high_plateforms environment for planning (just flat surfaces)

File: data/urdf/high_plateforms.urdf (robot description, URDF)
Before this commit: robot obstacle, 1 links, 0 joints
Links:
- link base_link: geometry collision mesh filename=package://hpp-rbprm-corba/meshes/high_plateforms_planning.s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; visual mesh filename=package://hpp-rbprm-corba/meshes/high_plateforms_planning.s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
