Commit message: Fix avNormal in generateContacts, modify envirs, skeleton and frog:
* add a torso box in frog trunk (so oriented fullbody torso has less risk to collide),
* shorten pelvis box of skeleton trunk,
* lower head DOF limits of frog (because animation not so nice),
* add frog on plateforms script (not used yet),
* re-orient plateform mesh (so characters have good starting orientation with 1,0,0,0),
* add database scripts for skeleton and frog,

File: data/urdf/frog/FrogLFootSphere.urdf (robot description, URDF)
Before this commit: robot FrogLFootSphere, 6 links, 5 joints
Joints:
- joint Head_rx: limit lower=-0.3 upper=0.3 effort=0 velocity=1.0 -> lower=-0.2 upper=0.2 effort=0 velocity=1.0
- joint Head_ry: limit lower=-0.3 upper=0.3 effort=0 velocity=1.0 -> lower=-0.2 upper=0.2 effort=0 velocity=1.0
- joint Head_rz: limit lower=-0.3 upper=0.3 effort=0 velocity=1.0 -> lower=-0.2 upper=0.2 effort=0 velocity=1.0

File: data/urdf/frog/FrogLHandSphere.urdf (robot description, URDF)
Before this commit: robot FrogLHandSphere, 6 links, 5 joints
Joints:
- joint Head_rx: limit lower=-0.3 upper=0.3 effort=0 velocity=1.0 -> lower=-0.2 upper=0.2 effort=0 velocity=1.0
- joint Head_ry: limit lower=-0.3 upper=0.3 effort=0 velocity=1.0 -> lower=-0.2 upper=0.2 effort=0 velocity=1.0
- joint Head_rz: limit lower=-0.3 upper=0.3 effort=0 velocity=1.0 -> lower=-0.2 upper=0.2 effort=0 velocity=1.0

File: data/urdf/frog/FrogRFootSphere.urdf (robot description, URDF)
Before this commit: robot FrogRFootSphere, 6 links, 5 joints
Joints:
- joint Head_rx: limit lower=-0.3 upper=0.3 effort=0 velocity=1.0 -> lower=-0.2 upper=0.2 effort=0 velocity=1.0
- joint Head_ry: limit lower=-0.3 upper=0.3 effort=0 velocity=1.0 -> lower=-0.2 upper=0.2 effort=0 velocity=1.0
- joint Head_rz: limit lower=-0.3 upper=0.3 effort=0 velocity=1.0 -> lower=-0.2 upper=0.2 effort=0 velocity=1.0

File: data/urdf/frog/FrogRHandSphere.urdf (robot description, URDF)
Before this commit: robot FrogRHandSphere, 6 links, 5 joints
Joints:
- joint Head_rx: limit lower=-0.3 upper=0.3 effort=0 velocity=1.0 -> lower=-0.2 upper=0.2 effort=0 velocity=1.0
- joint Head_ry: limit lower=-0.3 upper=0.3 effort=0 velocity=1.0 -> lower=-0.2 upper=0.2 effort=0 velocity=1.0
- joint Head_rz: limit lower=-0.3 upper=0.3 effort=0 velocity=1.0 -> lower=-0.2 upper=0.2 effort=0 velocity=1.0

File: data/urdf/frog/frog.urdf (robot description, URDF)
Before this commit: robot frog, 46 links, 45 joints
Joints:
- joint Head_rx: limit lower=-0.3 upper=0.3 effort=0 velocity=1.0 -> lower=-0.2 upper=0.2 effort=0 velocity=1.0
- joint Head_ry: limit lower=-0.3 upper=0.3 effort=0 velocity=1.0 -> lower=-0.2 upper=0.2 effort=0 velocity=1.0
- joint Head_rz: limit lower=-0.3 upper=0.3 effort=0 velocity=1.0 -> lower=-0.2 upper=0.2 effort=0 velocity=1.0
- joint LFoot_rz: limit lower=-0.5 upper=0.8 effort=0 velocity=1.0 -> lower=-1.3 upper=0.8 effort=0 velocity=1.0
- joint LHand_rx: limit lower=-0.3 upper=0.3 effort=0 velocity=1.0 -> lower=-0.45 upper=0.45 effort=0 velocity=1.0
- joint LShank_ry: limit lower=-0.3 upper=0.1 effort=0 velocity=1.0 -> lower=-0.3 upper=0.5 effort=0 velocity=1.0
- joint LShank_rz: limit lower=-0.8 upper=0.5 effort=0 velocity=1.0 -> lower=-0.8 upper=1.1 effort=0 velocity=1.0
- joint LThigh_rz: limit lower=-0.6 upper=0.2 effort=0 velocity=1.0 -> lower=-1.3 upper=0.2 effort=0 velocity=1.0
- joint RFoot_rz: limit lower=-0.8 upper=0.5 effort=0 velocity=1.0 -> lower=-0.8 upper=1.3 effort=0 velocity=1.0
- joint RHand_rx: limit lower=-0.3 upper=0.3 effort=0 velocity=1.0 -> lower=-0.45 upper=0.45 effort=0 velocity=1.0
- joint RShank_ry: limit lower=-0.3 upper=0.1 effort=0 velocity=1.0 -> lower=-0.3 upper=0.5 effort=0 velocity=1.0
- joint RShank_rz: limit lower=-0.5 upper=0.8 effort=0 velocity=1.0 -> lower=-1.1 upper=0.8 effort=0 velocity=1.0
- joint RThigh_rz: limit lower=-0.2 upper=0.6 effort=0 velocity=1.0 -> lower=-0.2 upper=1.3 effort=0 velocity=1.0

File: data/urdf/frog/frog_trunk.urdf (robot description, URDF)
Before this commit: robot frog_trunk, 5 links, 4 joints
Links:
- link Torso: geometry collision mesh filename=package://hpp-rbprm-corba/meshes/frog/Torso_box.stl; visual mesh filename=package://hpp-rbprm-corba/meshes/frog/Torso_view.dae
Joints:
- joint Head_rx: limit lower=-0.3 upper=0.3 effort=0 velocity=1.0 -> lower=-0.2 upper=0.2 effort=0 velocity=1.0
- joint Head_ry: limit lower=-0.3 upper=0.3 effort=0 velocity=1.0 -> lower=-0.2 upper=0.2 effort=0 velocity=1.0
- joint Head_rz: limit lower=-0.3 upper=0.3 effort=0 velocity=1.0 -> lower=-0.2 upper=0.2 effort=0 velocity=1.0
