Commit message: Add a head-box for the frog-trunk

File: data/urdf/frog/frog_trunk.urdf (robot description, URDF)
Before this commit: robot frog_trunk, 5 links, 4 joints
Links:
- link Head: geometry collision mesh filename=package://hpp-rbprm-corba/meshes/frog/Head_box.stl; visual mesh filename=package://hpp-rbprm-corba/meshes/frog/Head_view.dae
