Commit message: Add frog ROMs, improve spiderman extending pose

File: data/urdf/frog/frog.urdf (robot description, URDF)
Before this commit: robot frog, 45 links, 44 joints
Links:
- added link head_rom; visual mesh filename=package://hpp-rbprm-corba/meshes/frog/rhand_rom.stl
- link LHumerus: geometry collision mesh filename=package://hpp-rbprm-corba/meshes/frog/LHumerus.stl; visual mesh filename=package://hpp-rbprm-corba/meshes/frog/LHumerus.stl
- link RHumerus: geometry collision mesh filename=package://hpp-rbprm-corba/meshes/frog/RHumerus.stl; visual mesh filename=package://hpp-rbprm-corba/meshes/frog/RHumerus.stl
Joints:
- added joint head_rom_joint: type fixed, parent Head, child head_rom, origin xyz=0 0 0 rpy=0 0 0
- joint FrogLHandSphere: origin xyz=0.0184 -0.0116 -0.0103 rpy=0 0 0 -> xyz=0.0184 -0.0116 -0.0103 rpy=0 -0.1 0
- joint FrogRHandSphere: origin xyz=0.0169 0.0106 -0.0096 rpy=0 0 0 -> xyz=0.0169 0.0106 -0.0096 rpy=0 -0.1 0
- joint HeadRHumerus_J1: limit lower=-0.7 upper=0.7 effort=0 velocity=1.0 -> lower=-0.8 upper=0.8 effort=0 velocity=1.0
- joint HeadRHumerus_J2: limit lower=-0.7 upper=0.7 effort=0 velocity=1.0 -> lower=-0.8 upper=0.8 effort=0 velocity=1.0
- joint HumerusLForearm_J1: limit lower=-0.8 upper=0.8 effort=0 velocity=1.0 -> lower=-0.6 upper=0.6 effort=0 velocity=1.0
- joint HumerusLForearm_J2: limit lower=-0.8 upper=0.8 effort=0 velocity=1.0 -> lower=-0.6 upper=0.6 effort=0 velocity=1.0
- joint HumerusRForearm_J1: limit lower=-0.8 upper=0.8 effort=0 velocity=1.0 -> lower=-0.6 upper=0.6 effort=0 velocity=1.0
- joint HumerusRForearm_J2: limit lower=-0.8 upper=0.8 effort=0 velocity=1.0 -> lower=-0.6 upper=0.6 effort=0 velocity=1.0
- joint LFoot: limit lower=-0.3 upper=0.3 effort=0 velocity=1.0 -> lower=-0.5 upper=0.8 effort=0 velocity=1.0
- joint LShank: limit lower=-0.2 upper=0.2 effort=0 velocity=1.0 -> lower=-0.8 upper=0.5 effort=0 velocity=1.0
- joint LThigh: limit lower=-0.4 upper=0.4 effort=0 velocity=1.0 -> lower=-0.6 upper=0.2 effort=0 velocity=1.0
- joint RFoot: limit lower=-0.3 upper=0.3 effort=0 velocity=1.0 -> lower=-0.8 upper=0.5 effort=0 velocity=1.0
- joint RShank: limit lower=-0.2 upper=0.2 effort=0 velocity=1.0 -> lower=-0.5 upper=0.8 effort=0 velocity=1.0
- joint RThigh: limit lower=-0.4 upper=0.4 effort=0 velocity=1.0 -> lower=-0.2 upper=0.6 effort=0 velocity=1.0
- joint ShankLFoot_J1: limit lower=-0.3 upper=0.3 effort=0 velocity=1.0 -> lower=-0.4 upper=0.4 effort=0 velocity=1.0
- joint ShankLFoot_J2: limit lower=-0.3 upper=0.3 effort=0 velocity=1.0 -> lower=-0.2 upper=0.2 effort=0 velocity=1.0
- joint ShankRFoot_J1: limit lower=-0.3 upper=0.3 effort=0 velocity=1.0 -> lower=-0.4 upper=0.4 effort=0 velocity=1.0
- joint ShankRFoot_J2: limit lower=-0.3 upper=0.3 effort=0 velocity=1.0 -> lower=-0.2 upper=0.2 effort=0 velocity=1.0
- joint ThighLShank_J1: limit lower=-0.6 upper=0.6 effort=0 velocity=1.0 -> lower=-0.1 upper=0.1 effort=0 velocity=1.0
- joint ThighLShank_J2: limit lower=-0.6 upper=0.6 effort=0 velocity=1.0 -> lower=-0.3 upper=0.1 effort=0 velocity=1.0
- joint ThighRShank_J1: limit lower=-0.6 upper=0.6 effort=0 velocity=1.0 -> lower=-0.1 upper=0.1 effort=0 velocity=1.0
- joint ThighRShank_J2: limit lower=-0.6 upper=0.6 effort=0 velocity=1.0 -> lower=-0.3 upper=0.1 effort=0 velocity=1.0
- joint TorsoLThigh_J1: limit lower=-0.8 upper=0.8 effort=0 velocity=1.0 -> lower=-0.7 upper=0.7 effort=0 velocity=1.0
- joint TorsoLThigh_J2: limit lower=-0.8 upper=0.8 effort=0 velocity=1.0 -> lower=-0.9 upper=0.3 effort=0 velocity=1.0
- joint TorsoRThigh_J1: limit lower=-0.8 upper=0.8 effort=0 velocity=1.0 -> lower=-0.7 upper=0.7 effort=0 velocity=1.0
- joint TorsoRThigh_J2: limit lower=-0.8 upper=0.8 effort=0 velocity=1.0 -> lower=-0.9 upper=0.3 effort=0 velocity=1.0

File: data/urdf/spiderman/spiderman.urdf (robot description, URDF)
Before this commit: robot spiderman, 39 links, 38 joints
Links:
- removed link thorax_rhand_rom
Joints:
- removed joint thorax_rhand_rom_joint

Commit message: Improve leg limits of frog and change flexion config

File: data/urdf/frog/frog.urdf (robot description, URDF)
Before this commit: robot frog, 46 links, 45 joints
Joints:
- joint LFoot_rx: limit lower=-0.4 upper=0.4 effort=0 velocity=1.0 -> lower=-0.5 upper=0.2 effort=0 velocity=1.0
- joint LFoot_ry: limit lower=-0.2 upper=0.2 effort=0 velocity=1.0 -> lower=-0.2 upper=0.4 effort=0 velocity=1.0
- joint LFoot_rz: limit lower=-1.3 upper=0.8 effort=0 velocity=1.0 -> lower=-1.7 upper=0.5 effort=0 velocity=1.0
- joint LShank_rx: limit lower=-0.1 upper=0.1 effort=0 velocity=1.0 -> lower=-0.2 upper=0 effort=0 velocity=1.0
- joint LShank_ry: limit lower=-0.3 upper=0.5 effort=0 velocity=1.0 -> lower=-0.2 upper=0.6 effort=0 velocity=1.0
- joint LShank_rz: limit lower=-0.8 upper=1.1 effort=0 velocity=1.0 -> lower=-0.5 upper=1.2 effort=0 velocity=1.0
- joint LThigh_rx: limit lower=-0.7 upper=0.7 effort=0 velocity=1.0 -> lower=-0.5 upper=0 effort=0 velocity=1.0
- joint LThigh_ry: limit lower=-0.9 upper=0.3 effort=0 velocity=1.0 -> lower=-0.9 upper=0 effort=0 velocity=1.0
- joint LThigh_rz: limit lower=-1.3 upper=0.2 effort=0 velocity=1.0 -> lower=-1.4 upper=0.2 effort=0 velocity=1.0
- joint RFoot_rx: limit lower=-0.4 upper=0.4 effort=0 velocity=1.0 -> lower=-0.2 upper=0.5 effort=0 velocity=1.0
- joint RFoot_ry: limit lower=-0.2 upper=0.2 effort=0 velocity=1.0 -> lower=-0.4 upper=0.2 effort=0 velocity=1.0
- joint RFoot_rz: limit lower=-0.8 upper=1.3 effort=0 velocity=1.0 -> lower=-0.5 upper=1.7 effort=0 velocity=1.0
- joint RShank_rx: limit lower=-0.1 upper=0.1 effort=0 velocity=1.0 -> lower=0 upper=0.2 effort=0 velocity=1.0
- joint RShank_ry: limit lower=-0.3 upper=0.5 effort=0 velocity=1.0 -> lower=-0.2 upper=0.6 effort=0 velocity=1.0
- joint RShank_rz: limit lower=-1.1 upper=0.8 effort=0 velocity=1.0 -> lower=-1.2 upper=0.5 effort=0 velocity=1.0
- joint RThigh_rx: limit lower=-0.7 upper=0.7 effort=0 velocity=1.0 -> lower=0 upper=0.5 effort=0 velocity=1.0
- joint RThigh_ry: limit lower=-0.9 upper=0.3 effort=0 velocity=1.0 -> lower=-0.9 upper=0 effort=0 velocity=1.0
- joint RThigh_rz: limit lower=-0.2 upper=1.3 effort=0 velocity=1.0 -> lower=-0.2 upper=1.4 effort=0 velocity=1.0

Commit message: Try to improve frog benchmark:
* +0.2 to all jointBounds,
* bend frog L foot
* re-add shank-torso collision detection (very ugly collisions...)
* change database to 6_DOF
* TODO: bend frog R foot, adapt full-mesh...

File: data/urdf/frog/frog.urdf (robot description, URDF)
Before this commit: robot frog, 46 links, 45 joints
Joints:
- joint LFoot_rx: limit lower=-0.5 upper=0.2 effort=0 velocity=1.0 -> lower=-0.7 upper=0.4 effort=0 velocity=1.0
- joint LFoot_ry: limit lower=-0.2 upper=0.4 effort=0 velocity=1.0 -> lower=-0.4 upper=0.6 effort=0 velocity=1.0
- joint LFoot_rz: limit lower=-1.7 upper=0.5 effort=0 velocity=1.0 -> lower=-1.9 upper=0.7 effort=0 velocity=1.0
- joint LForearm_rx: limit lower=-0.6 upper=0.6 effort=0 velocity=1.0 -> lower=-0.8 upper=0.8 effort=0 velocity=1.0
- joint LForearm_ry: limit lower=-0.6 upper=0.6 effort=0 velocity=1.0 -> lower=-0.8 upper=0.8 effort=0 velocity=1.0
- joint LForearm_rz: limit lower=-0.5 upper=0.5 effort=0 velocity=1.0 -> lower=-0.7 upper=0.7 effort=0 velocity=1.0
- joint LHand_rx: limit lower=-0.45 upper=0.45 effort=0 velocity=1.0 -> lower=-0.65 upper=0.65 effort=0 velocity=1.0
- joint LHand_ry: limit lower=-0.3 upper=0.3 effort=0 velocity=1.0 -> lower=-0.5 upper=0.5 effort=0 velocity=1.0
- joint LHand_rz: limit lower=-0.3 upper=0.3 effort=0 velocity=1.0 -> lower=-0.5 upper=0.5 effort=0 velocity=1.0
- joint LHumerus_rx: limit lower=-0.7 upper=0.7 effort=0 velocity=1.0 -> lower=-0.9 upper=0.9 effort=0 velocity=1.0
- joint LHumerus_ry: limit lower=-0.7 upper=0.7 effort=0 velocity=1.0 -> lower=-0.9 upper=0.9 effort=0 velocity=1.0
- joint LHumerus_rz: limit lower=-0.4 upper=0.4 effort=0 velocity=1.0 -> lower=-0.6 upper=0.6 effort=0 velocity=1.0
- joint LShank_rx: limit lower=-0.2 upper=0 effort=0 velocity=1.0 -> lower=-0.4 upper=0.2 effort=0 velocity=1.0
- joint LShank_ry: limit lower=-0.2 upper=0.6 effort=0 velocity=1.0 -> lower=-0.4 upper=0.8 effort=0 velocity=1.0
- joint LShank_rz: limit lower=-0.5 upper=1.2 effort=0 velocity=1.0 -> lower=-0.7 upper=1.4 effort=0 velocity=1.0
- joint LThigh_rx: limit lower=-0.5 upper=0 effort=0 velocity=1.0 -> lower=-0.7 upper=0.2 effort=0 velocity=1.0
- joint LThigh_ry: limit lower=-0.9 upper=0 effort=0 velocity=1.0 -> lower=-1.1 upper=0.2 effort=0 velocity=1.0
- joint LThigh_rz: limit lower=-1.4 upper=0.2 effort=0 velocity=1.0 -> lower=-1.6 upper=0.4 effort=0 velocity=1.0
- joint RFoot_rx: limit lower=-0.2 upper=0.5 effort=0 velocity=1.0 -> lower=-0.4 upper=0.7 effort=0 velocity=1.0
- joint RFoot_ry: limit lower=-0.4 upper=0.2 effort=0 velocity=1.0 -> lower=-0.6 upper=0.4 effort=0 velocity=1.0
- joint RFoot_rz: limit lower=-0.5 upper=1.7 effort=0 velocity=1.0 -> lower=-0.7 upper=1.9 effort=0 velocity=1.0
- joint RForearm_rx: limit lower=-0.6 upper=0.6 effort=0 velocity=1.0 -> lower=-0.8 upper=0.8 effort=0 velocity=1.0
- joint RForearm_ry: limit lower=-0.6 upper=0.6 effort=0 velocity=1.0 -> lower=-0.8 upper=0.8 effort=0 velocity=1.0
- joint RForearm_rz: limit lower=-0.5 upper=0.5 effort=0 velocity=1.0 -> lower=-0.7 upper=0.7 effort=0 velocity=1.0
- joint RHand_rx: limit lower=-0.45 upper=0.45 effort=0 velocity=1.0 -> lower=-0.65 upper=0.65 effort=0 velocity=1.0
- joint RHand_ry: limit lower=-0.3 upper=0.3 effort=0 velocity=1.0 -> lower=-0.5 upper=0.5 effort=0 velocity=1.0
- joint RHand_rz: limit lower=-0.3 upper=0.3 effort=0 velocity=1.0 -> lower=-0.5 upper=0.5 effort=0 velocity=1.0
- joint RHumerus_rx: limit lower=-0.8 upper=0.8 effort=0 velocity=1.0 -> lower=-1 upper=1 effort=0 velocity=1.0
- joint RHumerus_ry: limit lower=-0.8 upper=0.8 effort=0 velocity=1.0 -> lower=-1 upper=1 effort=0 velocity=1.0
- joint RHumerus_rz: limit lower=-0.4 upper=0.4 effort=0 velocity=1.0 -> lower=-0.6 upper=0.6 effort=0 velocity=1.0
- joint RShank_rx: limit lower=0 upper=0.2 effort=0 velocity=1.0 -> lower=-0.2 upper=0.4 effort=0 velocity=1.0
- joint RShank_ry: limit lower=-0.2 upper=0.6 effort=0 velocity=1.0 -> lower=-0.4 upper=0.8 effort=0 velocity=1.0
- joint RShank_rz: limit lower=-1.2 upper=0.5 effort=0 velocity=1.0 -> lower=-1.4 upper=0.7 effort=0 velocity=1.0
- joint RThigh_rx: limit lower=0 upper=0.5 effort=0 velocity=1.0 -> lower=-0.2 upper=0.7 effort=0 velocity=1.0
- joint RThigh_ry: limit lower=-0.9 upper=0 effort=0 velocity=1.0 -> lower=-1.1 upper=0.2 effort=0 velocity=1.0
- joint RThigh_rz: limit lower=-0.2 upper=1.4 effort=0 velocity=1.0 -> lower=-0.4 upper=1.6 effort=0 velocity=1.0

Commit message: Add toe DOF to frog, and missing toe-changes in skeleton SRDF
TODO: adapt frog armature in blender file

File: data/urdf/frog/frog.urdf (robot description, URDF)
Before this commit: robot frog, 46 links, 45 joints
Links:
- added link LFootToe, mass 1; collision mesh filename=package://hpp-rbprm-corba/meshes/frog/LFootToe.stl; visual mesh filename=package://hpp-rbprm-corba/meshes/frog/LFootToe.stl
- added link RFootToe, mass 1; collision mesh filename=package://hpp-rbprm-corba/meshes/frog/RFootToe.stl; visual mesh filename=package://hpp-rbprm-corba/meshes/frog/RFootToe.stl
Joints:
- added joint LFootToe: type revolute, parent LFoot, child LFootToe, origin xyz=-0.0438 0.0852 -0.0153 rpy=0 0 0, axis 0 1 0, limit lower=-0.5 upper=0.5 effort=0 velocity=1.0
- added joint RFootToe: type revolute, parent RFoot, child RFootToe, origin xyz=-0.0473 -0.0954 -0.0172 rpy=0 0 0, axis 0 1 0, limit lower=-0.5 upper=0.5 effort=0 velocity=1.0
- joint FrogLFootSphere: origin xyz=-0.0436 0.0776 -0.032 rpy=0 0 0 -> xyz=-0.0016 0.0010 -0.0122 rpy=0 0 0; parent LFoot -> LFootToe
- joint FrogRFootSphere: origin xyz=-0.0461 -0.0853 -0.032 rpy=0 0 0 -> xyz=-0.0019 -0.0007 -0.0112 rpy=0 0 0; parent RFoot -> RFootToe
- joint LFoot_rz: limit lower=-1.9 upper=0.7 effort=0 velocity=1.0 -> lower=-1.9 upper=0.9 effort=0 velocity=1.0
- joint LShank_rz: limit lower=-0.7 upper=1.4 effort=0 velocity=1.0 -> lower=-1. upper=1.4 effort=0 velocity=1.0
- joint RFoot_rz: limit lower=-0.7 upper=1.9 effort=0 velocity=1.0 -> lower=-0.9 upper=1.9 effort=0 velocity=1.0
- joint RShank_rz: limit lower=-1.4 upper=0.7 effort=0 velocity=1.0 -> lower=-1.4 upper=1. effort=0 velocity=1.0

Commit message: Fix frog toe DOF name, roadmap-visibility-blender for IROS, minor changes in scripts

File: data/urdf/frog/frog.urdf (robot description, URDF)
Before this commit: robot frog, 48 links, 47 joints
Joints:
- removed joint LFootToe
- removed joint RFootToe
- added joint LFootToe_ry: type revolute, parent LFoot, child LFootToe, origin xyz=-0.0438 0.0852 -0.0153 rpy=0 0 0, axis 0 1 0, limit lower=-0.5 upper=0.5 effort=0 velocity=1.0
- added joint RFootToe_ry: type revolute, parent RFoot, child RFootToe, origin xyz=-0.0473 -0.0954 -0.0172 rpy=0 0 0, axis 0 1 0, limit lower=-0.5 upper=0.5 effort=0 velocity=1.0

Commit message: Change characters, envirs and scripts:
* for RB-trunk robots, replace meshes by boxes
* simplify the parkourWalls and high_plateforms for planning
* add hand-DOFs to jumperman, NOT TESTED YET
* fix some waypoint-paths in scripts

File: data/urdf/frog/frog.urdf (robot description, URDF)
Before this commit: robot frog, 48 links, 47 joints
Links:
- added link LHandFingers, mass 1; collision mesh filename=package://hpp-rbprm-corba/meshes/frog/LHandRHandFingers.stl; visual mesh filename=package://hpp-rbprm-corba/meshes/frog/LHandFingers.stl
- added link RHandFingers, mass 1; collision mesh filename=package://hpp-rbprm-corba/meshes/frog/RHandRHandFingers.stl; visual mesh filename=package://hpp-rbprm-corba/meshes/frog/RHandFingers.stl
- link Head: mass 2 -> 0
- link LFoot: mass 0.4 -> 1
- link LFootToe: mass 0.1 -> 1
- link LForearm: mass 0.5 -> 1
- link LHand: mass 0.3 -> 1
- link LHumerus: mass 0.8 -> 1
- link LShank: mass 0.6 -> 1
- link RFoot: mass 0.4 -> 1
- link RFootToe: mass 0.1 -> 1
- link RForearm: mass 0.5 -> 1
- link RHand: mass 0.3 -> 1
- link RHumerus: mass 0.8 -> 1
- link RShank: mass 0.6 -> 1
- link Torso: mass 4 -> 1
Joints:
- added joint FrogLHandFingers: type fixed, parent LHand, child FrogLHandFingers, origin xyz=0.0141 -0.0119 0.001 rpy=0 0 0
- added joint FrogRHandFingers: type fixed, parent RHand, child FrogRHandFingers, origin xyz=0.0134 0.0117 0.0018 rpy=0 0 0
- joint FrogLFootSphere: origin xyz=-0.0016 0.0010 -0.0122 rpy=0 0 0 -> xyz=-0.0016 0.0010 -0.013 rpy=0 0 0
- joint FrogLHandSphere: origin xyz=0.0184 -0.0116 -0.0103 rpy=0 -0.1 0 -> xyz=0.0059 -0.0038 -0.0137 rpy=0 0 0
- joint FrogRFootSphere: origin xyz=-0.0019 -0.0007 -0.0112 rpy=0 0 0 -> xyz=-0.0019 -0.0007 -0.013 rpy=0 0 0
- joint FrogRHandSphere: origin xyz=0.0169 0.0106 -0.0096 rpy=0 -0.1 0 -> xyz=0.007 0.0039 -0.0129 rpy=0 0 0

File: data/urdf/lamp/lamp.urdf (robot description, URDF)
Before this commit: robot lamp, 15 links, 14 joints
Links:
- removed link head_rom
Joints:
- removed joint head_rom_joint
- joint base_link_comshift_J: origin xyz=-0.023 0 0.245 rpy=0 0 0 -> xyz=0 0 0.1 rpy=0 0 0

File: data/urdf/lamp/lamp_trunk.urdf (robot description, URDF)
Before this commit: robot lamp_trunk, 5 links, 4 joints
Links:
- removed link head_rom
Joints:
- removed joint head_rom_joint
- joint base_link_comshift_J: origin xyz=-0.023 0 0.245 rpy=0 0 0 -> xyz=0 0 0.1 rpy=0 0 0

File: data/urdf/spiderman/spiderman.urdf (robot description, URDF)
Before this commit: robot spiderman, 41 links, 40 joints
Joints:
- joint SpidermanLHandSphere: origin xyz=-0.01 -0.0184 -0.04 rpy=0 0.2 -0.2 -> xyz=-0.0111 -0.0454 -0.0761 rpy=0 0 0
- joint SpidermanRHandSphere: origin xyz=-0.0 -0.0184 -0.06 rpy=0 0.2 -0.2 -> xyz=0.0152 -0.0559 -0.081 rpy=0 0 0

File: data/urdf/spiderman/spiderman_trunk.urdf (robot description, URDF)
Before this commit: robot spiderman_trunk, 8 links, 7 joints
Links:
- link Skull: geometry collision mesh filename=package://hpp-rbprm-corba/meshes/spiderman/spiderman-skull_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; visual mesh filename=package://hpp-rbprm-corba/meshes/spiderman/spiderman-skull_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

Commit message: Add frog masses

File: data/urdf/frog/frog.urdf (robot description, URDF)
Before this commit: robot frog, 50 links, 49 joints
Links:
- link Head: mass 0 -> 4.5
- link LFoot: mass 1 -> 0.2
- link LFootToe: mass 1 -> 0.1
- link LForearm: mass 1 -> 0.7
- link LHand: mass 1 -> 0.2
- link LHandFingers: mass 1 -> 0.1
- link LShank: mass 1 -> 0.7
- link RFoot: mass 1 -> 0.2
- link RFootToe: mass 1 -> 0.1
- link RForearm: mass 1 -> 0.7
- link RHand: mass 1 -> 0.2
- link RHandFingers: mass 1 -> 0.1
- link RShank: mass 1 -> 0.7
- link Torso: mass 1 -> 7.5
