Commit message: Add frog and new environment, fix Spiderman joint limits/directions and regenerate ROMs
* frog ROMs have not been generated yet !

File: data/urdf/spiderman/spiderman.urdf (robot description, URDF)
Before this commit: robot spiderman, 38 links, 37 joints
Links:
- removed link LFootSphere
- removed link LHandSphere
- removed link RFootSphere
- removed link RHandSphere
- added link SpidermanLFootSphere; collision sphere radius=0.01; visual sphere radius=0.01
- added link SpidermanLHandSphere; collision sphere radius=0.01; visual sphere radius=0.01
- added link SpidermanRFootSphere; collision sphere radius=0.01; visual sphere radius=0.01
- added link SpidermanRHandSphere; collision sphere radius=0.01; visual sphere radius=0.01
- added link thorax_rhand_rom; visual mesh filename=package://hpp-rbprm-corba/meshes/spiderman/rhand_rom.stl
Joints:
- removed joint LFootSphere
- removed joint LHandSphere
- removed joint RFootSphere
- removed joint RHandSphere
- added joint SpidermanLFootSphere: type fixed, parent LFoot, child SpidermanLFootSphere, origin xyz=0.00134 -0.16 -0.09568 rpy=0 0 0
- added joint SpidermanLHandSphere: type fixed, parent LHand, child SpidermanLHandSphere, origin xyz=-0.003 -0.0434 -0.0727 rpy=0 0.2 3.3415
- added joint SpidermanRFootSphere: type fixed, parent RFoot, child SpidermanRFootSphere, origin xyz=-0.00134 -0.16 -0.09568 rpy=0 0 0
- added joint SpidermanRHandSphere: type fixed, parent RHand, child SpidermanRHandSphere, origin xyz=0.0034 -0.0434 -0.0752 rpy=0 0.2 -0.2
- added joint thorax_rhand_rom_joint: type fixed, parent Thorax, child thorax_rhand_rom, origin xyz=0 0 0 rpy=0 0 0
- joint A_PelvisThorax_J1: axis 1 0 0 -> 0 -1 0
- joint A_ThoraxSkull_J1: axis 1 0 0 -> 0 -1 0
- joint LAnkle_J1: axis 0 1 0 -> 1 0 0; limit lower=-1.4 upper=1.4 effort=0 velocity=1.0 -> lower=-0.6 upper=1.1 effort=0 velocity=1.0
- joint LElbow_J1: axis 0 1 0 -> 1 0 0
- joint LHand: axis 1 0 0 -> 0 -1 0
- joint LHip_J1: axis 1 0 0 -> 0 -1 0; limit lower=-0.6 upper=1.3 effort=0 velocity=1.0 -> lower=-0.5 upper=1.1 effort=0 velocity=1.0
- joint LHip_J2: limit lower=-1.1 upper=1.4 effort=0 velocity=1.0 -> lower=-1.1 upper=1.3 effort=0 velocity=1.0
- joint LHumerus: axis 0 1 0 -> 1 0 0
- joint LShank: axis 0 1 0 -> 1 0 0; limit lower=-0.1 upper=2.5 effort=0 velocity=1.0 -> lower=-0.05 upper=1.9 effort=0 velocity=1.0
- joint LShoulder_J1: axis 1 0 0 -> 0 -1 0
- joint LThigh: axis 0 1 0 -> 1 0 0; limit lower=-2.6 upper=0.7 effort=0 velocity=1.0 -> lower=-2.5 upper=0.7 effort=0 velocity=1.0
- joint LWrist_J1: axis 0 1 0 -> 1 0 0
- joint RAnkle_J1: axis 0 1 0 -> 1 0 0; limit lower=-1.7 upper=1.7 effort=0 velocity=1.0 -> lower=-0.6 upper=1.1 effort=0 velocity=1.0
- joint RElbow_J1: axis 0 1 0 -> 0 -1 0
- joint RHand: axis 1 0 0 -> 0 -1 0
- joint RHip_J1: axis 1 0 0 -> 0 -1 0; limit lower=-1.3 upper=0.6 effort=0 velocity=1.0 -> lower=-1.1 upper=0.5 effort=0 velocity=1.0
- joint RHumerus: axis 0 1 0 -> 1 0 0
- joint RShank: axis 0 1 0 -> 1 0 0; limit lower=-0.05 upper=2.5 effort=0 velocity=1.0 -> lower=-0.05 upper=1.9 effort=0 velocity=1.0
- joint RShoulder_J1: axis 1 0 0 -> 0 -1 0
- joint RThigh: axis 0 1 0 -> 1 0 0; limit lower=-2.6 upper=0.9 effort=0 velocity=1.0 -> lower=-2.5 upper=0.7 effort=0 velocity=1.0
- joint RWrist_J1: axis 0 1 0 -> 1 0 0
- joint Skull: axis 0 1 0 -> 1 0 0
- joint Thorax: axis 0 1 0 -> 1 0 0

Commit message: reduce joint bound of spiderman thigh

File: data/urdf/spiderman/spiderman.urdf (robot description, URDF)
Before this commit: robot spiderman, 39 links, 38 joints
Joints:
- joint LThigh_ry: limit lower=-1.1 upper=0.5 effort=0 velocity=1.0 -> lower=-0.9 upper=0.3 effort=0 velocity=1.0
- joint LThigh_rz: limit lower=-1.1 upper=1.3 effort=0 velocity=1.0 -> lower=-0.2 upper=0.5 effort=0 velocity=1.0
- joint RThigh_ry: limit lower=-0.5 upper=1.1 effort=0 velocity=1.0 -> lower=-0.3 upper=0.9 effort=0 velocity=1.0
- joint RThigh_rz: limit lower=-1.3 upper=1.1 effort=0 velocity=1.0 -> lower=-0.2 upper=0.5 effort=0 velocity=1.0

Commit message: change some rotation axis in spiderman urdf in order to have symetry between limb (for reference pose)

File: data/urdf/spiderman/spiderman.urdf (robot description, URDF)
Before this commit: robot spiderman, 39 links, 38 joints
Joints:
- joint RForearm_rz: axis 0 0 1 -> 0 0 -1
- joint RHumerus_ry: axis 0 1 0 -> 0 -1 0; limit lower=-0.7 upper=2.4 effort=0 velocity=1.0 -> lower=-2.4 upper=0.7 effort=0 velocity=1.0
- joint RHumerus_rz: axis 0 0 1 -> 0 0 -1; limit lower=-1.4 upper=2.3 effort=0 velocity=1.0 -> lower=-2.1 upper=1.4 effort=0 velocity=1.0
- joint RThigh_ry: axis 0 1 0 -> 0 -1 0; limit lower=-0.3 upper=0.9 effort=0 velocity=1.0 -> lower=-0.9 upper=0.3 effort=0 velocity=1.0
- joint RThigh_rz: axis 0 0 1 -> 0 0 -1

Commit message: increase some joint bounds on spiderman

File: data/urdf/spiderman/spiderman.urdf (robot description, URDF)
Before this commit: robot spiderman, 39 links, 38 joints
Joints:
- joint LFoot_rx: limit lower=-0.6 upper=1.1 effort=0 velocity=1.0 -> lower=-0.8 upper=1.1 effort=0 velocity=1.0
- joint LShank_rx: limit lower=-0.05 upper=1.9 effort=0 velocity=1.0 -> lower=-0.05 upper=2.1 effort=0 velocity=1.0
- joint RFoot_rx: limit lower=-0.6 upper=1.1 effort=0 velocity=1.0 -> lower=-0.8 upper=1.1 effort=0 velocity=1.0
- joint RShank_rx: limit lower=-0.05 upper=1.9 effort=0 velocity=1.0 -> lower=-0.05 upper=2.1 effort=0 velocity=1.0

Commit message: small tweak in spiderman urdf for better 4-contact stance. Script for spiderman 4 contact OK

File: data/urdf/spiderman/spiderman.urdf (robot description, URDF)
Before this commit: robot spiderman, 39 links, 38 joints
Joints:
- joint LForearm_rz: limit lower=-3.3 upper=0.6 effort=0 velocity=1.0 -> lower=-2.3 upper=0.6 effort=0 velocity=1.0
- joint LHand_ry: limit lower=-0.5 upper=0.6 effort=0 velocity=1.0 -> lower=-0.6 upper=0.6 effort=0 velocity=1.0
- joint RForearm_rx: limit lower=-0.1 upper=2.9 effort=0 velocity=1.0 -> lower=-2.9 upper=0.1 effort=0 velocity=1.0
- joint RForearm_rz: limit lower=-0.6 upper=3.3 effort=0 velocity=1.0 -> lower=-2.3 upper=0.6 effort=0 velocity=1.0
- joint RHand_ry: axis 0 1 0 -> 0 -1 0; limit lower=-0.6 upper=0.5 effort=0 velocity=1.0 -> lower=-0.6 upper=0.6 effort=0 velocity=1.0
- joint SpidermanLFootSphere: origin xyz=0.00134 -0.1 -0.09568 rpy=0 0 0 -> xyz=0.00134 -0.17 -0.09568 rpy=0 0 0
- joint SpidermanLHandSphere: origin xyz=0 -0.0434 -0.08 rpy=0 0.2 3.3415 -> xyz=0.01 -0.0384 -0.07 rpy=0 0.2 -0.2
- joint SpidermanRFootSphere: origin xyz=-0.00134 -0.1 -0.09568 rpy=0 0 0 -> xyz=-0.00134 -0.17 -0.09568 rpy=0 0 0
- joint SpidermanRHandSphere: origin xyz=0 -0.0434 -0.08 rpy=0 0.2 -0.2 -> xyz=-0.01 -0.0384 -0.07 rpy=0 0.2 -0.2

Commit message: Add Foot Toe DOF for Spiderman
TODO: adapt Blender armature

File: data/urdf/spiderman/spiderman.urdf (robot description, URDF)
Before this commit: robot spiderman, 39 links, 38 joints
Links:
- added link LFootToe, mass 0.72029; collision mesh filename=package://hpp-rbprm-corba/meshes/spiderman/spiderman-LFootT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; visual mesh filename=package://hpp-rbprm-corba/meshes/spiderman/spiderman-LFootT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
- added link RFootToe, mass 0.72029; collision mesh filename=package://hpp-rbprm-corba/meshes/spiderman/spiderman-RFootT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; visual mesh filename=package://hpp-rbprm-corba/meshes/spiderman/spiderman-RFootT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
Joints:
- added joint LFootToe_rx: type revolute, parent LFoot, child LFootToe, origin xyz=0.0052 -0.1277 -0.0646 rpy=0 0 0, axis 1 0 0, limit lower=-0.7 upper=0.2 effort=0 velocity=1.0
- added joint RFootToe_rx: type revolute, parent RFoot, child RFootToe, origin xyz=-0.0047 -0.1259 -0.0639 rpy=0 0 0, axis 1 0 0, limit lower=-0.7 upper=0.2 effort=0 velocity=1.0
- joint SpidermanLFootSphere: origin xyz=0.00134 -0.1 -0.09568 rpy=0 0 0 -> xyz=-0.0001 -0.0229 -0.0306 rpy=0 0 0; parent LFoot -> LFootToe
- joint SpidermanRFootSphere: origin xyz=-0.00134 -0.1 -0.09568 rpy=0 0 0 -> xyz=0.0022 -0.0229 -0.0306 rpy=0 0 0; parent RFoot -> RFootToe

Commit message: change joint bounds in urdf and adapt script to new spiderman.urdf

File: data/urdf/spiderman/spiderman.urdf (robot description, URDF)
Before this commit: robot spiderman, 41 links, 40 joints
Joints:
- joint LFootToe_rx: limit lower=-0.7 upper=0.2 effort=0 velocity=1.0 -> lower=-1 upper=0.2 effort=0 velocity=1.0
- joint LFoot_rx: limit lower=-0.6 upper=1.1 effort=0 velocity=1.0 -> lower=-1.1 upper=1.1 effort=0 velocity=1.0
- joint LHand_ry: limit lower=-0.5 upper=0.6 effort=0 velocity=1.0 -> lower=-0.6 upper=0.6 effort=0 velocity=1.0
- joint LShank_rx: limit lower=-0.05 upper=1.9 effort=0 velocity=1.0 -> lower=-0.05 upper=2.4 effort=0 velocity=1.0
- joint LThigh_rz: limit lower=-0.2 upper=0.5 effort=0 velocity=1.0 -> lower=-0.4 upper=0.5 effort=0 velocity=1.0
- joint RFootToe_rx: limit lower=-0.7 upper=0.2 effort=0 velocity=1.0 -> lower=-1 upper=0.2 effort=0 velocity=1.0
- joint RFoot_rx: limit lower=-0.6 upper=1.1 effort=0 velocity=1.0 -> lower=-1.1 upper=1.1 effort=0 velocity=1.0
- joint RForearm_rx: limit lower=-0.1 upper=2.9 effort=0 velocity=1.0 -> lower=-2.9 upper=0.1 effort=0 velocity=1.0
- joint RForearm_rz: limit lower=-3.3 upper=0.6 effort=0 velocity=1.0 -> lower=-0.6 upper=3.3 effort=0 velocity=1.0
- joint RHand_ry: limit lower=-0.6 upper=0.5 effort=0 velocity=1.0 -> lower=-0.6 upper=0.6 effort=0 velocity=1.0
- joint RShank_rx: limit lower=-0.05 upper=1.9 effort=0 velocity=1.0 -> lower=-0.05 upper=2.4 effort=0 velocity=1.0
- joint RThigh_rz: limit lower=-0.5 upper=0.2 effort=0 velocity=1.0 -> lower=-0.5 upper=0.4 effort=0 velocity=1.0
- joint SpidermanLHandSphere: origin xyz=0 -0.0434 -0.08 rpy=0 0.2 3.3415 -> xyz=-0.01 -0.0184 -0.04 rpy=0 0.2 -0.2
- joint SpidermanRHandSphere: origin xyz=0 -0.0434 -0.08 rpy=0 0.2 -0.2 -> xyz=-0.0 -0.0184 -0.06 rpy=0 0.2 -0.2
