Commit message: Add bindings for parabola parameters (from hpp-corbaserver), spiderman modifs:
*split max velocity parameter (for parabola-SM) in takeoff and landing,
*renamed spiderman ROM urdf and srdf to avoid conflicts with the skeleton ones (installed
in the same folder)

File: data/urdf/spiderman/SpidermanLFootSphere.urdf (robot description, URDF)
Before this commit: robot RHandSphere, 9 links, 8 joints
Links:
- removed link thorax_rhand_rom
- added link pelvis_lfoot_rom; collision mesh filename=package://hpp-rbprm-corba/meshes/spiderman/lfoot_rom.stl; visual mesh filename=package://hpp-rbprm-corba/meshes/spiderman/lfoot_rom.stl
Joints:
- removed joint thorax_rhand_rom_joint
- added joint pelvis_lfoot_rom_joint: type fixed, parent Pelvis, child pelvis_lfoot_rom, origin xyz=0 0 0 rpy=0 0 0

File: data/urdf/spiderman/SpidermanRHandSphere.urdf (robot description, URDF)
Before this commit: robot LFootSphere, 9 links, 8 joints
Links:
- removed link pelvis_lfoot_rom
- added link thorax_rhand_rom; collision mesh filename=package://hpp-rbprm-corba/meshes/spiderman/rhand_rom.stl; visual mesh filename=package://hpp-rbprm-corba/meshes/spiderman/rhand_rom.stl
Joints:
- removed joint pelvis_lfoot_rom_joint
- added joint thorax_rhand_rom_joint: type fixed, parent Thorax, child thorax_rhand_rom, origin xyz=0 0 0 rpy=0 0 0

Commit message: Change Spiderman URDF and Blender (all joint in x-y-z order)
note: this breaks the symmetry

File: data/urdf/spiderman/SpidermanLFootSphere.urdf (robot description, URDF)
Before this commit: robot SpidermanLFootSphere, 9 links, 8 joints
Links:
- removed link Skull_rz
- removed link Thorax_rz
- added link Skull_rx
- added link Thorax_rx
Joints:
- removed joint A_Skull_ry
- removed joint A_Thorax_ry
- removed joint Skull_rx
- removed joint Thorax_rx
- added joint A_Skull_rx: type revolute, parent Thorax, child Skull_rx, origin xyz=-0.0006 0.0160 0.5204 rpy=0 0 0, axis 1 0 0, limit lower=-1.1 upper=0.6 effort=0 velocity=1.0
- added joint A_Thorax_rx: type revolute, parent Pelvis, child Thorax_rx, origin xyz=0.0006 -0.0373 0.0788 rpy=0 0 0, axis 1 0 0, limit lower=-0.8 upper=0.8 effort=0 velocity=1.0
- added joint Skull_ry: type revolute, parent Skull_rx, child Skull_ry, origin xyz=0 0 0 rpy=0 0 0, axis 0 1 0, limit lower=-0.3 upper=0.3 effort=0 velocity=1.0
- added joint Thorax_ry: type revolute, parent Thorax_rx, child Thorax_ry, origin xyz=0 0 0 rpy=0 0 0, axis 0 1 0, limit lower=-1 upper=1 effort=0 velocity=1.0
- joint Skull_rz: child Skull_rz -> Skull; limit lower=-1.4 upper=1.4 effort=0 velocity=1.0 -> lower=-1.4 upper=1. effort=0 velocity=1.0
- joint Thorax_rz: child Thorax_rz -> Thorax

File: data/urdf/spiderman/SpidermanLHandSphere.urdf (robot description, URDF)
Before this commit: robot SpidermanLHandSphere, 9 links, 8 joints
Links:
- removed link Skull_rz
- removed link Thorax_rz
- added link Skull_rx
- added link Thorax_rx
Joints:
- removed joint A_Skull_ry
- removed joint A_Thorax_ry
- removed joint Skull_rx
- removed joint Thorax_rx
- added joint A_Skull_rx: type revolute, parent Thorax, child Skull_rx, origin xyz=-0.0006 0.0160 0.5204 rpy=0 0 0, axis 1 0 0, limit lower=-1.1 upper=0.6 effort=0 velocity=1.0
- added joint A_Thorax_rx: type revolute, parent Pelvis, child Thorax_rx, origin xyz=0.0006 -0.0373 0.0788 rpy=0 0 0, axis 1 0 0, limit lower=-0.8 upper=0.8 effort=0 velocity=1.0
- added joint Skull_ry: type revolute, parent Skull_rx, child Skull_ry, origin xyz=0 0 0 rpy=0 0 0, axis 0 1 0, limit lower=-0.3 upper=0.3 effort=0 velocity=1.0
- added joint Thorax_ry: type revolute, parent Thorax_rx, child Thorax_ry, origin xyz=0 0 0 rpy=0 0 0, axis 0 1 0, limit lower=-1 upper=1 effort=0 velocity=1.0
- joint Skull_rz: child Skull_rz -> Skull; limit lower=-1.4 upper=1.4 effort=0 velocity=1.0 -> lower=-1.4 upper=1. effort=0 velocity=1.0
- joint Thorax_rz: child Thorax_rz -> Thorax

File: data/urdf/spiderman/SpidermanRFootSphere.urdf (robot description, URDF)
Before this commit: robot SpidermanRFootSphere, 9 links, 8 joints
Links:
- removed link Skull_rz
- removed link Thorax_rz
- added link Skull_rx
- added link Thorax_rx
Joints:
- removed joint A_Skull_ry
- removed joint A_Thorax_ry
- removed joint Skull_rx
- removed joint Thorax_rx
- added joint A_Skull_rx: type revolute, parent Thorax, child Skull_rx, origin xyz=-0.0006 0.0160 0.5204 rpy=0 0 0, axis 1 0 0, limit lower=-1.1 upper=0.6 effort=0 velocity=1.0
- added joint A_Thorax_rx: type revolute, parent Pelvis, child Thorax_rx, origin xyz=0.0006 -0.0373 0.0788 rpy=0 0 0, axis 1 0 0, limit lower=-0.8 upper=0.8 effort=0 velocity=1.0
- added joint Skull_ry: type revolute, parent Skull_rx, child Skull_ry, origin xyz=0 0 0 rpy=0 0 0, axis 0 1 0, limit lower=-0.3 upper=0.3 effort=0 velocity=1.0
- added joint Thorax_ry: type revolute, parent Thorax_rx, child Thorax_ry, origin xyz=0 0 0 rpy=0 0 0, axis 0 1 0, limit lower=-1 upper=1 effort=0 velocity=1.0
- joint Skull_rz: child Skull_rz -> Skull; limit lower=-1.4 upper=1.4 effort=0 velocity=1.0 -> lower=-1.4 upper=1. effort=0 velocity=1.0
- joint Thorax_rz: child Thorax_rz -> Thorax

File: data/urdf/spiderman/SpidermanRHandSphere.urdf (robot description, URDF)
Before this commit: robot SpidermanRHandSphere, 9 links, 8 joints
Links:
- removed link Skull_rz
- removed link Thorax_rz
- added link Skull_rx
- added link Thorax_rx
Joints:
- removed joint A_Skull_ry
- removed joint A_Thorax_ry
- removed joint Skull_rx
- removed joint Thorax_rx
- added joint A_Skull_rx: type revolute, parent Thorax, child Skull_rx, origin xyz=-0.0006 0.0160 0.5204 rpy=0 0 0, axis 1 0 0, limit lower=-1.1 upper=0.6 effort=0 velocity=1.0
- added joint A_Thorax_rx: type revolute, parent Pelvis, child Thorax_rx, origin xyz=0.0006 -0.0373 0.0788 rpy=0 0 0, axis 1 0 0, limit lower=-0.8 upper=0.8 effort=0 velocity=1.0
- added joint Skull_ry: type revolute, parent Skull_rx, child Skull_ry, origin xyz=0 0 0 rpy=0 0 0, axis 0 1 0, limit lower=-0.3 upper=0.3 effort=0 velocity=1.0
- added joint Thorax_ry: type revolute, parent Thorax_rx, child Thorax_ry, origin xyz=0 0 0 rpy=0 0 0, axis 0 1 0, limit lower=-1 upper=1 effort=0 velocity=1.0
- joint Skull_rz: child Skull_rz -> Skull; limit lower=-1.4 upper=1.4 effort=0 velocity=1.0 -> lower=-1.4 upper=1. effort=0 velocity=1.0
- joint Thorax_rz: child Thorax_rz -> Thorax

File: data/urdf/spiderman/spiderman.urdf (robot description, URDF)
Before this commit: robot spiderman, 39 links, 38 joints
Links:
- removed link LHumerus_rz
- removed link LThigh_rz
- removed link RHumerus_rz
- removed link RThigh_rz
- removed link Skull_rz
- removed link Thorax_rz
- added link LHumerus_rx
- added link LThigh_rx
- added link RHumerus_rx
- added link RThigh_rx
- added link Skull_rx
- added link Thorax_rx
Joints:
- removed joint A_Skull_ry
- removed joint A_Thorax_ry
- removed joint Skull_rx
- removed joint Thorax_rx
- added joint A_Skull_rx: type revolute, parent Thorax, child Skull_rx, origin xyz=-0.0006 0.0160 0.5204 rpy=0 0 0, axis 1 0 0, limit lower=-1.1 upper=0.6 effort=0 velocity=1.0
- added joint A_Thorax_rx: type revolute, parent Pelvis, child Thorax_rx, origin xyz=0.0006 -0.0373 0.0788 rpy=0 0 0, axis 1 0 0, limit lower=-0.8 upper=0.8 effort=0 velocity=1.0
- added joint Skull_ry: type revolute, parent Skull_rx, child Skull_ry, origin xyz=0 0 0 rpy=0 0 0, axis 0 1 0, limit lower=-0.3 upper=0.3 effort=0 velocity=1.0
- added joint Thorax_ry: type revolute, parent Thorax_rx, child Thorax_ry, origin xyz=0 0 0 rpy=0 0 0, axis 0 1 0, limit lower=-1 upper=1 effort=0 velocity=1.0
- joint LFoot_rx: limit lower=-0.8 upper=1.1 effort=0 velocity=1.0 -> lower=-0.6 upper=1.1 effort=0 velocity=1.0
- joint LForearm_rz: limit lower=-2.3 upper=0.6 effort=0 velocity=1.0 -> lower=-3.3 upper=0.6 effort=0 velocity=1.0
- joint LHand_ry: limit lower=-0.6 upper=0.6 effort=0 velocity=1.0 -> lower=-0.5 upper=0.6 effort=0 velocity=1.0
- joint LHumerus_rx: child LHumerus -> LHumerus_rx; origin xyz=0 0 0 rpy=0 0 0 -> xyz=0.1813 0.0529 0.3280 rpy=0 0 0; parent LHumerus_rz -> Thorax
- joint LHumerus_ry: origin xyz=0.1813 0.0529 0.3280 rpy=0 0 0 -> xyz=0 0 0 rpy=0 0 0; parent Thorax -> LHumerus_rx
- joint LHumerus_rz: child LHumerus_rz -> LHumerus
- joint LShank_rx: limit lower=-0.05 upper=2.1 effort=0 velocity=1.0 -> lower=-0.05 upper=1.9 effort=0 velocity=1.0
- joint LThigh_rx: child LThigh -> LThigh_rx; origin xyz=0 0 0 rpy=0 0 0 -> xyz=0.0908 -0.0355 -0.0850 rpy=0 0 0; parent LThigh_rz -> Pelvis
- joint LThigh_ry: origin xyz=0.0908 -0.0355 -0.0850 rpy=0 0 0 -> xyz=0 0 0 rpy=0 0 0; parent Pelvis -> LThigh_rx
- joint LThigh_rz: child LThigh_rz -> LThigh
- joint RFoot_rx: limit lower=-0.8 upper=1.1 effort=0 velocity=1.0 -> lower=-0.6 upper=1.1 effort=0 velocity=1.0
- joint RForearm_rx: limit lower=-2.9 upper=0.1 effort=0 velocity=1.0 -> lower=-0.1 upper=2.9 effort=0 velocity=1.0
- joint RForearm_rz: axis 0 0 -1 -> 0 0 1; limit lower=-2.3 upper=0.6 effort=0 velocity=1.0 -> lower=-3.3 upper=0.6 effort=0 velocity=1.0
- joint RHand_ry: axis 0 -1 0 -> 0 1 0; limit lower=-0.6 upper=0.6 effort=0 velocity=1.0 -> lower=-0.6 upper=0.5 effort=0 velocity=1.0
- joint RHumerus_rx: child RHumerus -> RHumerus_rx; origin xyz=0 0 0 rpy=0 0 0 -> xyz=-0.1938 0.0528 0.3355 rpy=0 0 0; parent RHumerus_rz -> Thorax
- joint RHumerus_ry: axis 0 -1 0 -> 0 1 0; limit lower=-2.4 upper=0.7 effort=0 velocity=1.0 -> lower=-0.7 upper=2.4 effort=0 velocity=1.0; origin xyz=-0.1938 0.0528 0.3355 rpy=0 0 0 -> xyz=0 0 0 rpy=0 0 0; parent Thorax -> RHumerus_rx
- joint RHumerus_rz: axis 0 0 -1 -> 0 0 1; child RHumerus_rz -> RHumerus; limit lower=-2.1 upper=1.4 effort=0 velocity=1.0 -> lower=-1.4 upper=2.1 effort=0 velocity=1.0
- joint RShank_rx: limit lower=-0.05 upper=2.1 effort=0 velocity=1.0 -> lower=-0.05 upper=1.9 effort=0 velocity=1.0
- joint RThigh_rx: child RThigh -> RThigh_rx; origin xyz=0 0 0 rpy=0 0 0 -> xyz=-0.0943 -0.0367 -0.0844 rpy=0 0 0; parent RThigh_rz -> Pelvis
- joint RThigh_ry: axis 0 -1 0 -> 0 1 0; limit lower=-0.9 upper=0.3 effort=0 velocity=1.0 -> lower=-0.3 upper=0.9 effort=0 velocity=1.0; origin xyz=-0.0943 -0.0367 -0.0844 rpy=0 0 0 -> xyz=0 0 0 rpy=0 0 0; parent Pelvis -> RThigh_rx
- joint RThigh_rz: axis 0 0 -1 -> 0 0 1; child RThigh_rz -> RThigh; limit lower=-0.2 upper=0.5 effort=0 velocity=1.0 -> lower=-0.5 upper=0.2 effort=0 velocity=1.0
- joint Skull_rz: child Skull_rz -> Skull; limit lower=-1.4 upper=1.4 effort=0 velocity=1.0 -> lower=-1.4 upper=1. effort=0 velocity=1.0
- joint SpidermanLFootSphere: origin xyz=0.00134 -0.17 -0.09568 rpy=0 0 0 -> xyz=0.00134 -0.1 -0.09568 rpy=0 0 0
- joint SpidermanLHandSphere: origin xyz=0.01 -0.0384 -0.07 rpy=0 0.2 -0.2 -> xyz=0 -0.0434 -0.08 rpy=0 0.2 3.3415
- joint SpidermanRFootSphere: origin xyz=-0.00134 -0.17 -0.09568 rpy=0 0 0 -> xyz=-0.00134 -0.1 -0.09568 rpy=0 0 0
- joint SpidermanRHandSphere: origin xyz=-0.01 -0.0384 -0.07 rpy=0 0.2 -0.2 -> xyz=0 -0.0434 -0.08 rpy=0 0.2 -0.2
- joint Thorax_rz: child Thorax_rz -> Thorax

File: data/urdf/spiderman/spiderman_trunk.urdf (robot description, URDF)
Before this commit: robot spiderman_trunk, 8 links, 7 joints
Links:
- removed link Skull_rz
- removed link Thorax_rz
- added link Skull_rx
- added link Thorax_rx
Joints:
- removed joint A_Skull_ry
- removed joint A_Thorax_ry
- removed joint Skull_rx
- removed joint Thorax_rx
- added joint A_Skull_rx: type revolute, parent Thorax, child Skull_rx, origin xyz=-0.0006 0.0160 0.5204 rpy=0 0 0, axis 1 0 0, limit lower=-1.1 upper=0.6 effort=0 velocity=1.0
- added joint A_Thorax_rx: type revolute, parent Pelvis, child Thorax_rx, origin xyz=0.0006 -0.0373 0.0788 rpy=0 0 0, axis 1 0 0, limit lower=-0.8 upper=0.8 effort=0 velocity=1.0
- added joint Skull_ry: type revolute, parent Skull_rx, child Skull_ry, origin xyz=0 0 0 rpy=0 0 0, axis 0 1 0, limit lower=-0.3 upper=0.3 effort=0 velocity=1.0
- added joint Thorax_ry: type revolute, parent Thorax_rx, child Thorax_ry, origin xyz=0 0 0 rpy=0 0 0, axis 0 1 0, limit lower=-1 upper=1 effort=0 velocity=1.0
- joint Skull_rz: child Skull_rz -> Skull; limit lower=-1.4 upper=1.4 effort=0 velocity=1.0 -> lower=-1.4 upper=1. effort=0 velocity=1.0
- joint Thorax_rz: child Thorax_rz -> Thorax

Commit message: Modify Jumperman mesh to fix hand orientations

File: data/urdf/spiderman/SpidermanLFootSphere.urdf (robot description, URDF)
Before this commit: robot SpidermanLFootSphere, 9 links, 8 joints
Joints:
- joint A_Skull_rx: limit lower=-1.1 upper=0.6 effort=0 velocity=1.0 -> lower=-0.3 upper=0.3 effort=0 velocity=1.0; origin xyz=-0.0006 0.0160 0.5204 rpy=0 0 0 -> xyz=0.0711 -0.0005 0.6039 rpy=0 0 0
- joint A_Thorax_rx: limit lower=-0.8 upper=0.8 effort=0 velocity=1.0 -> lower=-1 upper=1 effort=0 velocity=1.0; origin xyz=0.0006 -0.0373 0.0788 rpy=0 0 0 -> xyz=0.0373 0.0006 0.0788 rpy=0 0 0
- joint Skull_ry: limit lower=-0.3 upper=0.3 effort=0 velocity=1.0 -> lower=-1.1 upper=0.6 effort=0 velocity=1.0
- joint Thorax_ry: limit lower=-1 upper=1 effort=0 velocity=1.0 -> lower=-0.8 upper=0.8 effort=0 velocity=1.0
- joint base_link_J: origin xyz=0 0 0 rpy=0 0 1.57079632 -> xyz=0 0 0 rpy=0 0 0

File: data/urdf/spiderman/SpidermanLHandSphere.urdf (robot description, URDF)
Before this commit: robot SpidermanLHandSphere, 9 links, 8 joints
Joints:
- joint A_Skull_rx: limit lower=-1.1 upper=0.6 effort=0 velocity=1.0 -> lower=-0.3 upper=0.3 effort=0 velocity=1.0; origin xyz=-0.0006 0.0160 0.5204 rpy=0 0 0 -> xyz=0.0711 -0.0005 0.6039 rpy=0 0 0
- joint A_Thorax_rx: limit lower=-0.8 upper=0.8 effort=0 velocity=1.0 -> lower=-1 upper=1 effort=0 velocity=1.0; origin xyz=0.0006 -0.0373 0.0788 rpy=0 0 0 -> xyz=0.0373 0.0006 0.0788 rpy=0 0 0
- joint Skull_ry: limit lower=-0.3 upper=0.3 effort=0 velocity=1.0 -> lower=-1.1 upper=0.6 effort=0 velocity=1.0
- joint Thorax_ry: limit lower=-1 upper=1 effort=0 velocity=1.0 -> lower=-0.8 upper=0.8 effort=0 velocity=1.0
- joint base_link_J: origin xyz=0 0 0 rpy=0 0 1.57079632 -> xyz=0 0 0 rpy=0 0 0

File: data/urdf/spiderman/SpidermanRFootSphere.urdf (robot description, URDF)
Before this commit: robot SpidermanRFootSphere, 9 links, 8 joints
Joints:
- joint A_Skull_rx: limit lower=-1.1 upper=0.6 effort=0 velocity=1.0 -> lower=-0.3 upper=0.3 effort=0 velocity=1.0; origin xyz=-0.0006 0.0160 0.5204 rpy=0 0 0 -> xyz=0.0711 -0.0005 0.6039 rpy=0 0 0
- joint A_Thorax_rx: limit lower=-0.8 upper=0.8 effort=0 velocity=1.0 -> lower=-1 upper=1 effort=0 velocity=1.0; origin xyz=0.0006 -0.0373 0.0788 rpy=0 0 0 -> xyz=0.0373 0.0006 0.0788 rpy=0 0 0
- joint Skull_ry: limit lower=-0.3 upper=0.3 effort=0 velocity=1.0 -> lower=-1.1 upper=0.6 effort=0 velocity=1.0
- joint Thorax_ry: limit lower=-1 upper=1 effort=0 velocity=1.0 -> lower=-0.8 upper=0.8 effort=0 velocity=1.0
- joint base_link_J: origin xyz=0 0 0 rpy=0 0 1.57079632 -> xyz=0 0 0 rpy=0 0 0

File: data/urdf/spiderman/SpidermanRHandSphere.urdf (robot description, URDF)
Before this commit: robot SpidermanRHandSphere, 9 links, 8 joints
Joints:
- joint A_Skull_rx: limit lower=-1.1 upper=0.6 effort=0 velocity=1.0 -> lower=-0.3 upper=0.3 effort=0 velocity=1.0; origin xyz=-0.0006 0.0160 0.5204 rpy=0 0 0 -> xyz=0.0711 -0.0005 0.6039 rpy=0 0 0
- joint A_Thorax_rx: limit lower=-0.8 upper=0.8 effort=0 velocity=1.0 -> lower=-1 upper=1 effort=0 velocity=1.0; origin xyz=0.0006 -0.0373 0.0788 rpy=0 0 0 -> xyz=0.0373 0.0006 0.0788 rpy=0 0 0
- joint Skull_ry: limit lower=-0.3 upper=0.3 effort=0 velocity=1.0 -> lower=-1.1 upper=0.6 effort=0 velocity=1.0
- joint Thorax_ry: limit lower=-1 upper=1 effort=0 velocity=1.0 -> lower=-0.8 upper=0.8 effort=0 velocity=1.0
- joint base_link_J: origin xyz=0 0 0 rpy=0 0 1.57079632 -> xyz=0 0 0 rpy=0 0 0

File: data/urdf/spiderman/spiderman.urdf (robot description, URDF)
Before this commit: robot spiderman, 41 links, 40 joints
Links:
- removed link LFoot_rx
- removed link LForearm_rx
- removed link RFoot_rx
- removed link RForearm_rx
- added link LFoot_ry
- added link LForearm_ry
- added link RFoot_ry
- added link RForearm_ry
- link LFoot: mass 0.72029 -> 0.52
- link LFootToe: mass 0.72029 -> 0.2
- link RFoot: mass 0.72029 -> 0.52
- link RFootToe: mass 0.72029 -> 0.2
Joints:
- removed joint LFootToe_rx
- removed joint LFoot_rx
- removed joint LForearm_rx
- removed joint LShank_rx
- removed joint RFootToe_rx
- removed joint RFoot_rx
- removed joint RForearm_rx
- removed joint RShank_rx
- added joint LFootToe_ry: type revolute, parent LFoot, child LFootToe, origin xyz=0.1277 0.0052 -0.0646 rpy=0 0 0, axis 0 1 0, limit lower=-1 upper=0.2 effort=0 velocity=1.0
- added joint LFoot_ry: type revolute, parent LShank, child LFoot_ry, origin xyz=-0.0393 0.0026 -0.4117 rpy=0 0 0, axis 0 1 0, limit lower=-1.1 upper=1.1 effort=0 velocity=1.0
- added joint LForearm_ry: type revolute, parent LHumerus, child LForearm_ry, origin xyz=-0.0011 0.0454 -0.2573 rpy=0 0 0, axis 0 1 0, limit lower=-2.3 upper=0.01 effort=0 velocity=1.0
- added joint LShank_ry: type revolute, parent LThigh, child LShank, origin xyz=-0.0308 0 -0.4471 rpy=0 0 0, axis 0 1 0, limit lower=-0.05 upper=2.4 effort=0 velocity=1.0
- added joint RFootToe_ry: type revolute, parent RFoot, child RFootToe, origin xyz=0.1259 -0.0047 -0.0639 rpy=0 0 0, axis 0 1 0, limit lower=-1 upper=0.2 effort=0 velocity=1.0
- added joint RFoot_ry: type revolute, parent RShank, child RFoot_ry, origin xyz=-0.0310 0.0070 -0.4016 rpy=0 0 0, axis 0 1 0, limit lower=-1.1 upper=1.1 effort=0 velocity=1.0
- added joint RForearm_ry: type revolute, parent RHumerus, child RForearm_ry, origin xyz=0.0088 -0.0307 -0.2504 rpy=0 0 0, axis 0 1 0, limit lower=-2.3 upper=0.01 effort=0 velocity=1.0
- added joint RShank_ry: type revolute, parent RThigh, child RShank, origin xyz=-0.0385 0.0012 -0.4586 rpy=0 0 0, axis 0 1 0, limit lower=-0.05 upper=2.4 effort=0 velocity=1.0
- joint A_Skull_rx: limit lower=-1.1 upper=0.6 effort=0 velocity=1.0 -> lower=-0.3 upper=0.3 effort=0 velocity=1.0; origin xyz=-0.0006 0.0160 0.5204 rpy=0 0 0 -> xyz=0.0711 -0.0005 0.6039 rpy=0 0 0
- joint A_Thorax_rx: limit lower=-0.8 upper=0.8 effort=0 velocity=1.0 -> lower=-1 upper=1 effort=0 velocity=1.0; origin xyz=0.0006 -0.0373 0.0788 rpy=0 0 0 -> xyz=0.0373 0.0006 0.0788 rpy=0 0 0
- joint LFoot_rz: parent LFoot_rx -> LFoot_ry
- joint LForearm_rz: limit lower=-3.3 upper=0.6 effort=0 velocity=1.0 -> lower=-1.6 upper=1.7 effort=0 velocity=1.0; parent LForearm_rx -> LForearm_ry
- joint LHand_rx: limit lower=-1.6 upper=1.4 effort=0 velocity=1.0 -> lower=-1.4 upper=1.6 effort=0 velocity=1.0; origin xyz=0.1986 -0.0758 -0.1368 rpy=0 0 0 -> xyz=0.0351 0.0088 -0.2751 rpy=0 0 0
- joint LHumerus_rx: limit lower=-2.9 upper=0.7 effort=0 velocity=1.0 -> lower=-0.3 upper=2.3 effort=0 velocity=1.0; origin xyz=0.1813 0.0529 0.3280 rpy=0 0 0 -> xyz=-0.0467 0.1854 0.3285 rpy=0 0 0
- joint LHumerus_ry: limit lower=-2.4 upper=0.7 effort=0 velocity=1.0 -> lower=-2.8 upper=1.6 effort=0 velocity=1.0
- joint LHumerus_rz: limit lower=-2.1 upper=1.4 effort=0 velocity=1.0 -> lower=-1.5 upper=1.5 effort=0 velocity=1.0
- joint LThigh_rx: limit lower=-2.5 upper=0.7 effort=0 velocity=1.0 -> lower=-1.2 upper=1.5 effort=0 velocity=1.0; origin xyz=0.0908 -0.0355 -0.0850 rpy=0 0 0 -> xyz=0.0355 0.0908 -0.0850 rpy=0 0 0
- joint LThigh_ry: limit lower=-0.9 upper=0.3 effort=0 velocity=1.0 -> lower=-2.5 upper=0.7 effort=0 velocity=1.0
- joint LThigh_rz: limit lower=-0.4 upper=0.5 effort=0 velocity=1.0 -> lower=-1.2 upper=1.6 effort=0 velocity=1.0
- joint RFoot_rz: parent RFoot_rx -> RFoot_ry
- joint RForearm_rz: limit lower=-0.6 upper=3.3 effort=0 velocity=1.0 -> lower=-1.7 upper=1.6 effort=0 velocity=1.0; parent RForearm_rx -> RForearm_ry
- joint RHand_rx: origin xyz=-0.1949 -0.0716 -0.1326 rpy=0 0 0 -> xyz=0.038 -0.0018 -0.2731 rpy=0 0 0
- joint RHumerus_rx: limit lower=-2.9 upper=0.7 effort=0 velocity=1.0 -> lower=-2.3 upper=0.3 effort=0 velocity=1.0; origin xyz=-0.1938 0.0528 0.3355 rpy=0 0 0 -> xyz=-0.0467 -0.1906 0.3285 rpy=0 0 0
- joint RHumerus_ry: limit lower=-0.7 upper=2.4 effort=0 velocity=1.0 -> lower=-2.8 upper=1.6 effort=0 velocity=1.0
- joint RHumerus_rz: limit lower=-1.4 upper=2.1 effort=0 velocity=1.0 -> lower=-1.5 upper=1.5 effort=0 velocity=1.0
- joint RThigh_rx: limit lower=-2.5 upper=0.7 effort=0 velocity=1.0 -> lower=-1.6 upper=1.2 effort=0 velocity=1.0; origin xyz=-0.0943 -0.0367 -0.0844 rpy=0 0 0 -> xyz=0.0367 -0.0943 -0.0844 rpy=0 0 0
- joint RThigh_ry: limit lower=-0.3 upper=0.9 effort=0 velocity=1.0 -> lower=-2.5 upper=0.7 effort=0 velocity=1.0
- joint RThigh_rz: limit lower=-0.5 upper=0.4 effort=0 velocity=1.0 -> lower=-1.6 upper=1.2 effort=0 velocity=1.0
- joint Skull_ry: limit lower=-0.3 upper=0.3 effort=0 velocity=1.0 -> lower=-1.1 upper=0.6 effort=0 velocity=1.0
- joint SpidermanLFootSphere: origin xyz=-0.0001 -0.0229 -0.0306 rpy=0 0 0 -> xyz=0.0229 -0.0001 -0.0306 rpy=0 0 0
- joint SpidermanLHandSphere: origin xyz=-0.0111 -0.0454 -0.0761 rpy=0 0 0 -> xyz=0.021 -0.0589 -0.0591 rpy=0 0 0
- joint SpidermanRFootSphere: origin xyz=0.0022 -0.0229 -0.0306 rpy=0 0 0 -> xyz=0.0229 0.0022 -0.0306 rpy=0 0 0
- joint SpidermanRHandSphere: origin xyz=0.0152 -0.0559 -0.081 rpy=0 0 0 -> xyz=0.0183 0.0517 -0.0678 rpy=0 0 0
- joint Thorax_ry: limit lower=-1 upper=1 effort=0 velocity=1.0 -> lower=-0.8 upper=0.8 effort=0 velocity=1.0
- joint base_link_J: origin xyz=0 0 0 rpy=0 0 1.57079632 -> xyz=0 0 0 rpy=0 0 0

File: data/urdf/spiderman/spiderman_trunk.urdf (robot description, URDF)
Before this commit: robot spiderman_trunk, 8 links, 7 joints
Links:
- added link pelvis_lfoot_rom; visual mesh filename=package://hpp-rbprm-corba/meshes/spiderman/lfoot_rom.stl
- added link pelvis_rfoot_rom; visual mesh filename=package://hpp-rbprm-corba/meshes/spiderman/rfoot_rom.stl
- added link thorax_lhand_rom; visual mesh filename=package://hpp-rbprm-corba/meshes/spiderman/lhand_rom.stl
- added link thorax_rhand_rom; visual mesh filename=package://hpp-rbprm-corba/meshes/spiderman/rhand_rom.stl
Joints:
- added joint pelvis_lfoot_rom_joint: type fixed, parent Pelvis, child pelvis_lfoot_rom, origin xyz=0 0 0 rpy=0 0 0
- added joint pelvis_rfoot_rom_joint: type fixed, parent Pelvis, child pelvis_rfoot_rom, origin xyz=0 0 0 rpy=0 0 0
- added joint thorax_lhand_rom_joint: type fixed, parent Thorax, child thorax_lhand_rom, origin xyz=0 0 0 rpy=0 0 0
- added joint thorax_rhand_rom_joint: type fixed, parent Thorax, child thorax_rhand_rom, origin xyz=0 0 0 rpy=0 0 0
- joint A_Skull_rx: limit lower=-1.1 upper=0.6 effort=0 velocity=1.0 -> lower=-0.3 upper=0.3 effort=0 velocity=1.0; origin xyz=-0.0006 0.0160 0.5204 rpy=0 0 0 -> xyz=0.0711 -0.0005 0.6039 rpy=0 0 0
- joint A_Thorax_rx: limit lower=-0.8 upper=0.8 effort=0 velocity=1.0 -> lower=-1 upper=1 effort=0 velocity=1.0; origin xyz=0.0006 -0.0373 0.0788 rpy=0 0 0 -> xyz=0.0373 0.0006 0.0788 rpy=0 0 0
- joint Skull_ry: limit lower=-0.3 upper=0.3 effort=0 velocity=1.0 -> lower=-1.1 upper=0.6 effort=0 velocity=1.0
- joint Thorax_ry: limit lower=-1 upper=1 effort=0 velocity=1.0 -> lower=-0.8 upper=0.8 effort=0 velocity=1.0
- joint base_link_J: origin xyz=0 0 0 rpy=0 0 1.57079632 -> xyz=0 0 0 rpy=0 0 0
