Commit message: Change ref configs of armlessSkeleton (and joint limits)

File: data/urdf/ant/ant_trunk.urdf (robot description, URDF)
Before this commit: robot ant_trunk, 12 links, 11 joints
Links:
- link Abdomen: geometry collision mesh filename=package://hpp-rbprm-corba/meshes/ant/Abdomen_box.stl; visual mesh filename=package://hpp-rbprm-corba/meshes/ant/Abdomen_box.stl
- link Head: geometry collision mesh filename=package://hpp-rbprm-corba/meshes/ant/Skull_box.stl; visual mesh filename=package://hpp-rbprm-corba/meshes/ant/Skull_box.stl

File: data/urdf/skeleton/armlessSkeleton.urdf (robot description, URDF)
Before this commit: robot armlessSkeleton, 42 links, 41 joints
Joints:
- joint LAnkle_J1: limit lower=-1.2 upper=1.2 effort=0 velocity=1.0 -> lower=-1.4 upper=1.2 effort=0 velocity=1.0
- joint LShank: limit lower=-0.05 upper=2.3 effort=0 velocity=1.0 -> lower=-0.05 upper=2.4 effort=0 velocity=1.0
- joint RAnkle_J1: limit lower=-1.2 upper=1.2 effort=0 velocity=1.0 -> lower=-1.4 upper=1.2 effort=0 velocity=1.0
- joint RShank: limit lower=-0.05 upper=2.3 effort=0 velocity=1.0 -> lower=-0.05 upper=2.4 effort=0 velocity=1.0
