Commit message: Add skeleton and ant meshes, do not use boxes in fullbody URDF

File: data/urdf/ant/ant.urdf (robot description, URDF)
Before this commit: robot articulated_ant, 80 links, 79 joints
Links:
- link Abdomen: geometry collision mesh filename=package://hpp-rbprm-corba/meshes/ant/Abdomen.stl; visual mesh filename=package://hpp-rbprm-corba/meshes/ant/Abdomen.stl
- link Head: geometry collision mesh filename=package://hpp-rbprm-corba/meshes/ant/Skull.stl; visual mesh filename=package://hpp-rbprm-corba/meshes/ant/Skull.stl
- link Thorax: geometry collision mesh filename=package://hpp-rbprm-corba/meshes/ant/Thorax.stl; visual mesh filename=package://hpp-rbprm-corba/meshes/ant/Thorax.stl

Commit message: Fix pelvis box mesh of Spiderman, remove spheres in SRDF files (no collision field)

File: data/urdf/ant/ant.urdf (robot description, URDF)
Before this commit: robot articulated_ant, 80 links, 79 joints
Links:
- added link virtualThorax
Joints:
- added joint virtualThorax: type fixed, parent base_link, child virtualThorax, origin xyz=0 0 0 rpy=0 0 0

File: data/urdf/frog/frog.urdf (robot description, URDF)
Before this commit: robot frog, 45 links, 44 joints
Links:
- added link virtualTorso
Joints:
- added joint virtualTorso: type fixed, parent base_link, child virtualTorso, origin xyz=0 0 0 rpy=0 0 0
- joint FrogLFootSphere: origin xyz=-0.0436 0.0776 -0.0269 rpy=0 0 0 -> xyz=-0.0436 0.0776 -0.032 rpy=0 0 0
- joint FrogRFootSphere: origin xyz=-0.0461 -0.0853 -0.0268 rpy=0 0 0 -> xyz=-0.0461 -0.0853 -0.032 rpy=0 0 0

File: data/urdf/spiderman/spiderman.urdf (robot description, URDF)
Before this commit: robot spiderman, 38 links, 37 joints
Links:
- added link virtualPelvis
Joints:
- added joint virtualPelvis: type fixed, parent base_link, child virtualPelvis, origin xyz=0 0 0 rpy=0 0 0

Commit message: save changes in scripts and urdfs

File: data/urdf/ant/ant.urdf (robot description, URDF)
Before this commit: robot articulated_ant, 73 links, 72 joints
Links:
- link LBShank: geometry visual mesh filename=package://hpp-rbprm-corba/meshes/ant/LBShank.stl
Joints:
- joint LBThigh_ry: limit lower=-1 upper=1 effort=0 velocity=1.0 -> lower=-1 upper=1.1 effort=0 velocity=1.0

File: data/urdf/cave.urdf (robot description, URDF)
Before this commit: robot obstacle, 1 links, 0 joints
Links:
- link base_link: geometry collision mesh filename=package://hpp-rbprm-corba/meshes/cave.stl; visual mesh filename=package://hpp-rbprm-corba/meshes/cave.stl

Commit message: Update scripts, undo urdf changes

File: data/urdf/ant/ant.urdf (robot description, URDF)
Before this commit: robot articulated_ant, 73 links, 72 joints
Links:
- link LBShank: geometry collision mesh filename=package://hpp-rbprm-corba/meshes/ant/LBShank.stl; visual mesh filename=package://hpp-rbprm-corba/meshes/ant/LBShank.stl
Joints:
- joint LBThigh_ry: limit lower=-1 upper=1.1 effort=0 velocity=1.0 -> lower=-1 upper=1 effort=0 velocity=1.0

Commit message: Fix ant joint limits according to (fixed) extending pose

File: data/urdf/ant/ant.urdf (robot description, URDF)
Before this commit: robot articulated_ant, 73 links, 72 joints
Joints:
- joint LBThigh_ry: limit lower=-1 upper=1 effort=0 velocity=1.0 -> lower=-1 upper=1.2 effort=0 velocity=1.0
- joint LFThigh_ry: limit lower=-1 upper=1 effort=0 velocity=1.0 -> lower=-1 upper=1.2 effort=0 velocity=1.0
- joint LMThigh_ry: limit lower=-1 upper=1 effort=0 velocity=1.0 -> lower=-1 upper=1.2 effort=0 velocity=1.0
- joint RBShank_ry: limit lower=-1 upper=1 effort=0 velocity=1.0 -> lower=-1.2 upper=1 effort=0 velocity=1.0
- joint RBThigh_ry: limit lower=-1 upper=1 effort=0 velocity=1.0 -> lower=-1.2 upper=1 effort=0 velocity=1.0
- joint RFShank_ry: limit lower=-1 upper=1 effort=0 velocity=1.0 -> lower=-1.2 upper=1 effort=0 velocity=1.0
- joint RFThigh_ry: limit lower=-1 upper=1 effort=0 velocity=1.0 -> lower=-1.2 upper=1 effort=0 velocity=1.0
- joint RMShank_ry: limit lower=-1 upper=1 effort=0 velocity=1.0 -> lower=-1.2 upper=1 effort=0 velocity=1.0
- joint RMThigh_ry: limit lower=-1 upper=1 effort=0 velocity=1.0 -> lower=-1.2 upper=1 effort=0 velocity=1.0

Commit message: Add parkour_walls envir, add masses in URDFs, shift geom origin of lamp toward COM

File: data/urdf/ant/ant.urdf (robot description, URDF)
Before this commit: robot articulated_ant, 73 links, 72 joints
Links:
- link Abdomen: mass 0 -> 1.5
- link Head: mass 4.2276 -> 1.3
- link LAntena: mass 1 -> 0.05
- link LAntenaFoot: mass 1 -> 0.05
- link LBFoot: mass 1 -> 0.1
- link LBShank: mass 1 -> 0.2
- link LBThigh: mass 1 -> 0.3
- link LFFoot: mass 1 -> 0.1
- link LFShank: mass 1 -> 0.2
- link LFThigh: mass 1 -> 0.3
- link LMFoot: mass 1 -> 0.1
- link LMShank: mass 1 -> 0.2
- link LMThigh: mass 1 -> 0.3
- link RAntena: mass 1 -> 0.05
- link RAntenaFoot: mass 1 -> 0.05
- link RBFoot: mass 1 -> 0.1
- link RBShank: mass 1 -> 0.2
- link RBThigh: mass 1 -> 0.3
- link RFFoot: mass 1 -> 0.1
- link RFShank: mass 1 -> 0.2
- link RFThigh: mass 1 -> 0.3
- link RMFoot: mass 1 -> 0.1
- link RMShank: mass 1 -> 0.2
- link RMThigh: mass 1 -> 0.3
- link Thorax: mass 1 -> 2

File: data/urdf/frog/frog.urdf (robot description, URDF)
Before this commit: robot frog, 48 links, 47 joints
Links:
- link Head: mass 0 -> 2
- link LFoot: mass 1 -> 0.4
- link LFootToe: mass 1 -> 0.1
- link LForearm: mass 1 -> 0.5
- link LHand: mass 1 -> 0.3
- link LHumerus: mass 1 -> 0.8
- link LShank: mass 1 -> 0.6
- link RFoot: mass 1 -> 0.4
- link RFootToe: mass 1 -> 0.1
- link RForearm: mass 1 -> 0.5
- link RHand: mass 1 -> 0.3
- link RHumerus: mass 1 -> 0.8
- link RShank: mass 1 -> 0.6
- link Torso: mass 1 -> 4

File: data/urdf/lamp/lamp.urdf (robot description, URDF)
Before this commit: robot lamp, 14 links, 13 joints
Links:
- removed link head_rom
- added link base_link_comshift
Joints:
- removed joint head_rom_joint
- added joint base_link_comshift_J: type fixed, parent base_link_comshift, child Head, origin xyz=-0.023 0 0.245 rpy=0 0 0
- joint base_link_J: child Head -> base_link_comshift

Commit message: Adapt to modifs in hpp-rbprm, add contact-ref config for ant database:
* fix timed-ballistic-path for arbitrary number of subpath in each parabola,
* add boolean to choose to use flexion pose while computing contacts (for DOF not contacting),
* add function to store velocities and theta in fullbody, to check if convexCone from new contacts
 makes the trajectory satisfying non-sliding constraint,
* add parameter to set if generateContact fills the state from the fullbody computation or
directly from the configuration datas (e.g. position of end-effector, contact status harcoded
to true)
* ant_test_interp script has been updated with these changes, NOT the other scripts

File: data/urdf/ant/ant.urdf (robot description, URDF)
Before this commit: robot articulated_ant, 73 links, 72 joints
Joints:
- joint LBFoot_rx: limit lower=-0.2 upper=0.2 effort=0 velocity=1.0 -> lower=-0.4 upper=0.2 effort=0 velocity=1.0
- joint LBShank_rx: axis (none) -> 1 0 0; limit (none) -> lower=-0.7 upper=0.7 effort=0 velocity=1.0; type fixed -> revolute
- joint LBShank_ry: limit lower=-1 upper=1 effort=0 velocity=1.0 -> lower=-1.2 upper=1.2 effort=0 velocity=1.0
- joint LBThigh_ry: limit lower=-1 upper=1.2 effort=0 velocity=1.0 -> lower=-1.2 upper=1.2 effort=0 velocity=1.0
- joint LFShank_rx: axis (none) -> 1 0 0; limit (none) -> lower=-0.7 upper=0.7 effort=0 velocity=1.0; type fixed -> revolute
- joint LFShank_ry: limit lower=-1 upper=1 effort=0 velocity=1.0 -> lower=-1.2 upper=1.2 effort=0 velocity=1.0
- joint LFThigh_ry: limit lower=-1 upper=1.2 effort=0 velocity=1.0 -> lower=-1.2 upper=1.2 effort=0 velocity=1.0
- joint LMShank_rx: axis (none) -> 1 0 0; limit (none) -> lower=-0.7 upper=0.7 effort=0 velocity=1.0; type fixed -> revolute
- joint LMShank_ry: limit lower=-1 upper=1 effort=0 velocity=1.0 -> lower=-1.2 upper=1.2 effort=0 velocity=1.0
- joint LMThigh_ry: limit lower=-1 upper=1.2 effort=0 velocity=1.0 -> lower=-1.2 upper=1.2 effort=0 velocity=1.0
- joint RBFoot_rx: limit lower=-0.2 upper=0.2 effort=0 velocity=1.0 -> lower=-0.4 upper=0.2 effort=0 velocity=1.0
- joint RBShank_rx: axis (none) -> 1 0 0; limit (none) -> lower=-0.7 upper=0.7 effort=0 velocity=1.0; type fixed -> revolute
- joint RBShank_ry: limit lower=-1.2 upper=1 effort=0 velocity=1.0 -> lower=-1.2 upper=1.2 effort=0 velocity=1.0
- joint RBThigh_ry: limit lower=-1.2 upper=1 effort=0 velocity=1.0 -> lower=-1.2 upper=1.2 effort=0 velocity=1.0
- joint RFFoot_rx: limit lower=-0.2 upper=0.2 effort=0 velocity=1.0 -> lower=-0.4 upper=0.2 effort=0 velocity=1.0
- joint RFShank_rx: axis (none) -> 1 0 0; limit (none) -> lower=-0.7 upper=0.7 effort=0 velocity=1.0; type fixed -> revolute
- joint RFShank_ry: limit lower=-1.2 upper=1 effort=0 velocity=1.0 -> lower=-1.2 upper=1.2 effort=0 velocity=1.0
- joint RFThigh_ry: limit lower=-1.2 upper=1 effort=0 velocity=1.0 -> lower=-1.2 upper=1.2 effort=0 velocity=1.0
- joint RMShank_rx: axis (none) -> 1 0 0; limit (none) -> lower=-0.7 upper=0.7 effort=0 velocity=1.0; type fixed -> revolute
- joint RMShank_ry: limit lower=-1.2 upper=1 effort=0 velocity=1.0 -> lower=-1.2 upper=1.2 effort=0 velocity=1.0
- joint RMThigh_ry: limit lower=-1.2 upper=1 effort=0 velocity=1.0 -> lower=-1.2 upper=1.2 effort=0 velocity=1.0
