Commit message: Fix ant URDFs orientations, add contactSize and setPose (not tested yet)

File: data/urdf/ant/LBFootSphere.urdf (robot description, URDF)
Before this commit: robot LBFootSphere, 21 links, 20 joints
Joints:
- joint base_link_J: origin xyz=0.001 -0.0382 -0.1982 rpy=0 0 0 -> xyz=0.001 -0.0382 -0.1982 rpy=0 0 1.570796

File: data/urdf/ant/LFFootSphere.urdf (robot description, URDF)
Before this commit: robot LFFootSphere, 21 links, 20 joints
Joints:
- joint base_link_J: origin xyz=0.001 -0.0382 -0.1982 rpy=0 0 0 -> xyz=0.001 -0.0382 -0.1982 rpy=0 0 1.570796

File: data/urdf/ant/LMFootSphere.urdf (robot description, URDF)
Before this commit: robot LMFootSphere, 21 links, 20 joints
Joints:
- joint base_link_J: origin xyz=0.001 -0.0382 -0.1982 rpy=0 0 0 -> xyz=0.001 -0.0382 -0.1982 rpy=0 0 1.570796

File: data/urdf/ant/RBFootSphere.urdf (robot description, URDF)
Before this commit: robot RBFootSphere, 21 links, 20 joints
Joints:
- joint base_link_J: origin xyz=0.001 -0.0382 -0.1982 rpy=0 0 0 -> xyz=0.001 -0.0382 -0.1982 rpy=0 0 1.570796

File: data/urdf/ant/RFFootSphere.urdf (robot description, URDF)
Before this commit: robot RFFootSphere, 21 links, 20 joints
Joints:
- joint base_link_J: origin xyz=0.001 -0.0382 -0.1982 rpy=0 0 0 -> xyz=0.001 -0.0382 -0.1982 rpy=0 0 1.570796

File: data/urdf/ant/RMFootSphere.urdf (robot description, URDF)
Before this commit: robot RMFootSphere, 21 links, 20 joints
Joints:
- joint base_link_J: origin xyz=0.001 -0.0382 -0.1982 rpy=0 0 0 -> xyz=0.001 -0.0382 -0.1982 rpy=0 0 1.570796

File: data/urdf/ant/ant.urdf (robot description, URDF)
Before this commit: robot articulated_ant, 80 links, 79 joints
Joints:
- joint LBFoot: limit lower=-0.1 upper=0.1 effort=0 velocity=1.0 -> lower=-0.2 upper=0.2 effort=0 velocity=1.0
- joint LBShank: limit lower=-0.1 upper=0.1 effort=0 velocity=1.0 -> lower=-0.8 upper=0.8 effort=0 velocity=1.0
- joint LBThigh: limit lower=-0.5 upper=0.5 effort=0 velocity=1.0 -> lower=-0.7 upper=0.7 effort=0 velocity=1.0
- joint LFFoot: limit lower=-0.1 upper=0.1 effort=0 velocity=1.0 -> lower=-0.2 upper=0.2 effort=0 velocity=1.0
- joint LFShank: limit lower=-0.1 upper=0.1 effort=0 velocity=1.0 -> lower=-0.8 upper=0.8 effort=0 velocity=1.0
- joint LFThigh: limit lower=-0.5 upper=0.5 effort=0 velocity=1.0 -> lower=-0.7 upper=0.7 effort=0 velocity=1.0
- joint LMFoot: limit lower=-0.1 upper=0.1 effort=0 velocity=1.0 -> lower=-0.2 upper=0.2 effort=0 velocity=1.0
- joint LMShank: limit lower=-0.1 upper=0.1 effort=0 velocity=1.0 -> lower=-0.8 upper=0.8 effort=0 velocity=1.0
- joint LMThigh: limit lower=-0.5 upper=0.5 effort=0 velocity=1.0 -> lower=-0.7 upper=0.7 effort=0 velocity=1.0
- joint RBFoot: limit lower=-0.1 upper=0.1 effort=0 velocity=1.0 -> lower=-0.2 upper=0.2 effort=0 velocity=1.0
- joint RBShank: limit lower=-0.1 upper=0.1 effort=0 velocity=1.0 -> lower=-0.8 upper=0.8 effort=0 velocity=1.0
- joint RBThigh: limit lower=-0.5 upper=0.5 effort=0 velocity=1.0 -> lower=-0.7 upper=0.7 effort=0 velocity=1.0
- joint RFFoot: limit lower=-0.1 upper=0.1 effort=0 velocity=1.0 -> lower=-0.2 upper=0.2 effort=0 velocity=1.0
- joint RFShank: limit lower=-0.1 upper=0.1 effort=0 velocity=1.0 -> lower=-0.8 upper=0.8 effort=0 velocity=1.0
- joint RFThigh: limit lower=-0.5 upper=0.5 effort=0 velocity=1.0 -> lower=-0.7 upper=0.7 effort=0 velocity=1.0
- joint RMFoot: limit lower=-0.1 upper=0.1 effort=0 velocity=1.0 -> lower=-0.2 upper=0.2 effort=0 velocity=1.0
- joint RMShank: limit lower=-0.1 upper=0.1 effort=0 velocity=1.0 -> lower=-0.8 upper=0.8 effort=0 velocity=1.0
- joint RMThigh: limit lower=-0.5 upper=0.5 effort=0 velocity=1.0 -> lower=-0.7 upper=0.7 effort=0 velocity=1.0
- joint ThoraxLBFoot_J2: axis (none) -> 0 1 0; limit (none) -> lower=-0.4 upper=0.4 effort=0 velocity=1.0; type fixed -> revolute
- joint ThoraxLBShank_J2: limit lower=-0.8 upper=0.8 effort=0 velocity=1.0 -> lower=-1 upper=1 effort=0 velocity=1.0
- joint ThoraxLBThigh_J1: limit lower=-0.2 upper=0.2 effort=0 velocity=1.0 -> lower=-1.2 upper=1.2 effort=0 velocity=1.0
- joint ThoraxLBThigh_J2: limit lower=-0.8 upper=0.8 effort=0 velocity=1.0 -> lower=-1 upper=1 effort=0 velocity=1.0
- joint ThoraxLFFoot_J1: limit lower=-0.2 upper=0.2 effort=0 velocity=1.0 -> lower=-0.4 upper=0.4 effort=0 velocity=1.0
- joint ThoraxLFFoot_J2: axis (none) -> 0 1 0; limit (none) -> lower=-0.2 upper=0.2 effort=0 velocity=1.0; type fixed -> revolute
- joint ThoraxLFShank_J2: limit lower=-0.8 upper=0.8 effort=0 velocity=1.0 -> lower=-1 upper=1 effort=0 velocity=1.0
- joint ThoraxLFThigh_J1: limit lower=-0.2 upper=0.2 effort=0 velocity=1.0 -> lower=-1.2 upper=1.2 effort=0 velocity=1.0
- joint ThoraxLFThigh_J2: limit lower=-0.8 upper=0.8 effort=0 velocity=1.0 -> lower=-1 upper=1 effort=0 velocity=1.0
- joint ThoraxLMFoot_J2: axis (none) -> 0 1 0; limit (none) -> lower=-0.4 upper=0.4 effort=0 velocity=1.0; type fixed -> revolute
- joint ThoraxLMShank_J2: limit lower=-0.8 upper=0.8 effort=0 velocity=1.0 -> lower=-1 upper=1 effort=0 velocity=1.0
- joint ThoraxLMThigh_J1: limit lower=-0.2 upper=0.2 effort=0 velocity=1.0 -> lower=-1.2 upper=1.2 effort=0 velocity=1.0
- joint ThoraxLMThigh_J2: limit lower=-0.8 upper=0.8 effort=0 velocity=1.0 -> lower=-1 upper=1 effort=0 velocity=1.0
- joint ThoraxRBFoot_J2: axis (none) -> 0 1 0; limit (none) -> lower=-0.4 upper=0.4 effort=0 velocity=1.0; type fixed -> revolute
- joint ThoraxRBShank_J2: limit lower=-0.8 upper=0.8 effort=0 velocity=1.0 -> lower=-1 upper=1 effort=0 velocity=1.0
- joint ThoraxRBThigh_J1: limit lower=-0.2 upper=0.2 effort=0 velocity=1.0 -> lower=-1.2 upper=1.2 effort=0 velocity=1.0
- joint ThoraxRBThigh_J2: limit lower=-0.8 upper=0.8 effort=0 velocity=1.0 -> lower=-1 upper=1 effort=0 velocity=1.0
- joint ThoraxRFFoot_J2: axis (none) -> 0 1 0; limit (none) -> lower=-0.4 upper=0.4 effort=0 velocity=1.0; type fixed -> revolute
- joint ThoraxRFShank_J2: limit lower=-0.8 upper=0.8 effort=0 velocity=1.0 -> lower=-1 upper=1 effort=0 velocity=1.0
- joint ThoraxRFThigh_J1: limit lower=-0.2 upper=0.2 effort=0 velocity=1.0 -> lower=-1.2 upper=1.2 effort=0 velocity=1.0
- joint ThoraxRFThigh_J2: limit lower=-0.8 upper=0.8 effort=0 velocity=1.0 -> lower=-1 upper=1 effort=0 velocity=1.0
- joint ThoraxRMFoot_J2: axis (none) -> 0 1 0; limit (none) -> lower=-0.4 upper=0.4 effort=0 velocity=1.0; type fixed -> revolute
- joint ThoraxRMShank_J2: limit lower=-0.8 upper=0.8 effort=0 velocity=1.0 -> lower=-1 upper=1 effort=0 velocity=1.0
- joint ThoraxRMThigh_J1: limit lower=-0.2 upper=0.2 effort=0 velocity=1.0 -> lower=-1.2 upper=1.2 effort=0 velocity=1.0
- joint ThoraxRMThigh_J2: limit lower=-0.8 upper=0.8 effort=0 velocity=1.0 -> lower=-1 upper=1 effort=0 velocity=1.0
- joint base_link_J: origin xyz=0.001 -0.0382 -0.1982 rpy=0 0 0 -> xyz=0.001 -0.0382 -0.1982 rpy=0 0 1.570796

File: data/urdf/ant/ant_trunk.urdf (robot description, URDF)
Before this commit: robot ant_trunk, 20 links, 19 joints
Joints:
- joint base_link_J: origin xyz=0.001 -0.0382 -0.1982 rpy=0 0 0 -> xyz=0.001 -0.0382 -0.1982 rpy=0 0 1.570796

Commit message: Fix URDFs, update scripts to new URDFs, increase cave size

File: data/urdf/ant/LBFootSphere.urdf (robot description, URDF)
Before this commit: robot LBFootSphere, 21 links, 20 joints
Links:
- removed link HeadRAntena_rx
- removed link HeadRAntena_ry
- added link RAntena_rx
- added link RAntena_ry
Joints:
- removed joint AntenaFoot_rx
- removed joint AntenaFoot_ry
- removed joint Antena_rx
- removed joint Antena_ry
- added joint LAntenaFoot_rx: type revolute, parent LAntena, child LAntenaFoot_rx, origin xyz=0.0267 -0.0198 0.1006 rpy=0 0 0, axis 1 0 0, limit lower=-0.4 upper=0.4 effort=0 velocity=1.0
- added joint LAntenaFoot_ry: type revolute, parent LAntenaFoot_rx, child LAntenaFoot_ry, origin xyz=0 0 0 rpy=0 0 0, axis 0 1 0, limit lower=-0.4 upper=0.4 effort=0 velocity=1.0
- added joint LAntena_rx: type revolute, parent Head, child LAntena_rx, origin xyz=0.0176 -0.1027 0.0225 rpy=0 0 0, axis 1 0 0, limit lower=-0.4 upper=0.4 effort=0 velocity=1.0
- added joint LAntena_ry: type revolute, parent LAntena_rx, child LAntena_ry, origin xyz=0 0 0 rpy=0 0 0, axis 0 1 0, limit lower=-0.4 upper=0.4 effort=0 velocity=1.0
- joint LAntenaFoot_rz: parent AntenaFoot_ry -> LAntenaFoot_ry
- joint LAntena_rz: parent Antena_ry -> LAntena_ry

File: data/urdf/ant/LFFootSphere.urdf (robot description, URDF)
Before this commit: robot LFFootSphere, 21 links, 20 joints
Links:
- removed link HeadRAntena_rx
- removed link HeadRAntena_ry
- added link RAntena_rx
- added link RAntena_ry
Joints:
- removed joint AntenaFoot_rx
- removed joint AntenaFoot_ry
- removed joint Antena_rx
- removed joint Antena_ry
- added joint LAntenaFoot_rx: type revolute, parent LAntena, child LAntenaFoot_rx, origin xyz=0.0267 -0.0198 0.1006 rpy=0 0 0, axis 1 0 0, limit lower=-0.4 upper=0.4 effort=0 velocity=1.0
- added joint LAntenaFoot_ry: type revolute, parent LAntenaFoot_rx, child LAntenaFoot_ry, origin xyz=0 0 0 rpy=0 0 0, axis 0 1 0, limit lower=-0.4 upper=0.4 effort=0 velocity=1.0
- added joint LAntena_rx: type revolute, parent Head, child LAntena_rx, origin xyz=0.0176 -0.1027 0.0225 rpy=0 0 0, axis 1 0 0, limit lower=-0.4 upper=0.4 effort=0 velocity=1.0
- added joint LAntena_ry: type revolute, parent LAntena_rx, child LAntena_ry, origin xyz=0 0 0 rpy=0 0 0, axis 0 1 0, limit lower=-0.4 upper=0.4 effort=0 velocity=1.0
- joint LAntenaFoot_rz: parent AntenaFoot_ry -> LAntenaFoot_ry
- joint LAntena_rz: parent Antena_ry -> LAntena_ry

File: data/urdf/ant/LMFootSphere.urdf (robot description, URDF)
Before this commit: robot LMFootSphere, 21 links, 20 joints
Links:
- removed link HeadRAntena_rx
- removed link HeadRAntena_ry
- added link RAntena_rx
- added link RAntena_ry
Joints:
- removed joint AntenaFoot_rx
- removed joint AntenaFoot_ry
- removed joint Antena_rx
- removed joint Antena_ry
- added joint LAntenaFoot_rx: type revolute, parent LAntena, child LAntenaFoot_rx, origin xyz=0.0267 -0.0198 0.1006 rpy=0 0 0, axis 1 0 0, limit lower=-0.4 upper=0.4 effort=0 velocity=1.0
- added joint LAntenaFoot_ry: type revolute, parent LAntenaFoot_rx, child LAntenaFoot_ry, origin xyz=0 0 0 rpy=0 0 0, axis 0 1 0, limit lower=-0.4 upper=0.4 effort=0 velocity=1.0
- added joint LAntena_rx: type revolute, parent Head, child LAntena_rx, origin xyz=0.0176 -0.1027 0.0225 rpy=0 0 0, axis 1 0 0, limit lower=-0.4 upper=0.4 effort=0 velocity=1.0
- added joint LAntena_ry: type revolute, parent LAntena_rx, child LAntena_ry, origin xyz=0 0 0 rpy=0 0 0, axis 0 1 0, limit lower=-0.4 upper=0.4 effort=0 velocity=1.0
- joint LAntenaFoot_rz: parent AntenaFoot_ry -> LAntenaFoot_ry
- joint LAntena_rz: parent Antena_ry -> LAntena_ry

File: data/urdf/ant/RBFootSphere.urdf (robot description, URDF)
Before this commit: robot RBFootSphere, 21 links, 20 joints
Links:
- removed link HeadRAntena_rx
- removed link HeadRAntena_ry
- added link RAntena_rx
- added link RAntena_ry
Joints:
- removed joint AntenaFoot_rx
- removed joint AntenaFoot_ry
- removed joint Antena_rx
- removed joint Antena_ry
- added joint LAntenaFoot_rx: type revolute, parent LAntena, child LAntenaFoot_rx, origin xyz=0.0267 -0.0198 0.1006 rpy=0 0 0, axis 1 0 0, limit lower=-0.4 upper=0.4 effort=0 velocity=1.0
- added joint LAntenaFoot_ry: type revolute, parent LAntenaFoot_rx, child LAntenaFoot_ry, origin xyz=0 0 0 rpy=0 0 0, axis 0 1 0, limit lower=-0.4 upper=0.4 effort=0 velocity=1.0
- added joint LAntena_rx: type revolute, parent Head, child LAntena_rx, origin xyz=0.0176 -0.1027 0.0225 rpy=0 0 0, axis 1 0 0, limit lower=-0.4 upper=0.4 effort=0 velocity=1.0
- added joint LAntena_ry: type revolute, parent LAntena_rx, child LAntena_ry, origin xyz=0 0 0 rpy=0 0 0, axis 0 1 0, limit lower=-0.4 upper=0.4 effort=0 velocity=1.0
- joint LAntenaFoot_rz: parent AntenaFoot_ry -> LAntenaFoot_ry
- joint LAntena_rz: parent Antena_ry -> LAntena_ry

File: data/urdf/ant/RFFootSphere.urdf (robot description, URDF)
Before this commit: robot RFFootSphere, 21 links, 20 joints
Links:
- removed link HeadRAntena_rx
- removed link HeadRAntena_ry
- added link RAntena_rx
- added link RAntena_ry
Joints:
- removed joint AntenaFoot_rx
- removed joint AntenaFoot_ry
- removed joint Antena_rx
- removed joint Antena_ry
- added joint LAntenaFoot_rx: type revolute, parent LAntena, child LAntenaFoot_rx, origin xyz=0.0267 -0.0198 0.1006 rpy=0 0 0, axis 1 0 0, limit lower=-0.4 upper=0.4 effort=0 velocity=1.0
- added joint LAntenaFoot_ry: type revolute, parent LAntenaFoot_rx, child LAntenaFoot_ry, origin xyz=0 0 0 rpy=0 0 0, axis 0 1 0, limit lower=-0.4 upper=0.4 effort=0 velocity=1.0
- added joint LAntena_rx: type revolute, parent Head, child LAntena_rx, origin xyz=0.0176 -0.1027 0.0225 rpy=0 0 0, axis 1 0 0, limit lower=-0.4 upper=0.4 effort=0 velocity=1.0
- added joint LAntena_ry: type revolute, parent LAntena_rx, child LAntena_ry, origin xyz=0 0 0 rpy=0 0 0, axis 0 1 0, limit lower=-0.4 upper=0.4 effort=0 velocity=1.0
- joint LAntenaFoot_rz: parent AntenaFoot_ry -> LAntenaFoot_ry
- joint LAntena_rz: parent Antena_ry -> LAntena_ry

File: data/urdf/ant/RMFootSphere.urdf (robot description, URDF)
Before this commit: robot RMFootSphere, 21 links, 20 joints
Links:
- removed link HeadRAntena_rx
- removed link HeadRAntena_ry
- added link RAntena_rx
- added link RAntena_ry
Joints:
- removed joint AntenaFoot_rx
- removed joint AntenaFoot_ry
- removed joint Antena_rx
- removed joint Antena_ry
- added joint LAntenaFoot_rx: type revolute, parent LAntena, child LAntenaFoot_rx, origin xyz=0.0267 -0.0198 0.1006 rpy=0 0 0, axis 1 0 0, limit lower=-0.4 upper=0.4 effort=0 velocity=1.0
- added joint LAntenaFoot_ry: type revolute, parent LAntenaFoot_rx, child LAntenaFoot_ry, origin xyz=0 0 0 rpy=0 0 0, axis 0 1 0, limit lower=-0.4 upper=0.4 effort=0 velocity=1.0
- added joint LAntena_rx: type revolute, parent Head, child LAntena_rx, origin xyz=0.0176 -0.1027 0.0225 rpy=0 0 0, axis 1 0 0, limit lower=-0.4 upper=0.4 effort=0 velocity=1.0
- added joint LAntena_ry: type revolute, parent LAntena_rx, child LAntena_ry, origin xyz=0 0 0 rpy=0 0 0, axis 0 1 0, limit lower=-0.4 upper=0.4 effort=0 velocity=1.0
- joint LAntenaFoot_rz: parent AntenaFoot_ry -> LAntenaFoot_ry
- joint LAntena_rz: parent Antena_ry -> LAntena_ry

File: data/urdf/ant/ant.urdf (robot description, URDF)
Before this commit: robot articulated_ant, 80 links, 79 joints
Links:
- removed link AntenaFoot_rx
- removed link AntenaFoot_ry
- added link LAntenaFoot_rx
- added link LAntenaFoot_ry
Joints:
- removed joint AntenaFoot_rx
- removed joint AntenaFoot_ry
- removed joint Antena_rx
- removed joint Antena_ry
- added joint LAntenaFoot_rx: type revolute, parent LAntena, child LAntenaFoot_rx, origin xyz=0.0267 -0.0198 0.1006 rpy=0 0 0, axis 1 0 0, limit lower=-0.4 upper=0.4 effort=0 velocity=1.0
- added joint LAntenaFoot_ry: type revolute, parent LAntenaFoot_rx, child LAntenaFoot_ry, origin xyz=0 0 0 rpy=0 0 0, axis 0 1 0, limit lower=-0.4 upper=0.4 effort=0 velocity=1.0
- added joint LAntena_rx: type revolute, parent Head, child LAntena_rx, origin xyz=0.0176 -0.1027 0.0225 rpy=0 0 0, axis 1 0 0, limit lower=-0.4 upper=0.4 effort=0 velocity=1.0
- added joint LAntena_ry: type revolute, parent LAntena_rx, child LAntena_ry, origin xyz=0 0 0 rpy=0 0 0, axis 0 1 0, limit lower=-0.4 upper=0.4 effort=0 velocity=1.0
- joint LAntenaFoot_rz: parent AntenaFoot_ry -> LAntenaFoot_ry
- joint LAntena_rz: parent Antena_ry -> LAntena_ry

File: data/urdf/ant/ant_trunk.urdf (robot description, URDF)
Before this commit: robot ant_trunk, 20 links, 19 joints
Joints:
- removed joint AntenaFoot_rx
- removed joint AntenaFoot_ry
- removed joint Antena_rx
- removed joint Antena_ry
- added joint LAntenaFoot_rx: type revolute, parent LAntena, child LAntenaFoot_rx, origin xyz=0.0267 -0.0198 0.1006 rpy=0 0 0, axis 1 0 0, limit lower=-0.4 upper=0.4 effort=0 velocity=1.0
- added joint LAntenaFoot_ry: type revolute, parent LAntenaFoot_rx, child LAntenaFoot_ry, origin xyz=0 0 0 rpy=0 0 0, axis 0 1 0, limit lower=-0.4 upper=0.4 effort=0 velocity=1.0
- added joint LAntena_rx: type revolute, parent Head, child LAntena_rx, origin xyz=0.0176 -0.1027 0.0225 rpy=0 0 0, axis 1 0 0, limit lower=-0.4 upper=0.4 effort=0 velocity=1.0
- added joint LAntena_ry: type revolute, parent LAntena_rx, child LAntena_ry, origin xyz=0 0 0 rpy=0 0 0, axis 0 1 0, limit lower=-0.4 upper=0.4 effort=0 velocity=1.0
- joint LAntenaFoot_rz: parent AntenaFoot_ry -> LAntenaFoot_ry
- joint LAntena_rz: parent Antena_ry -> LAntena_ry

File: data/urdf/frog/frog.urdf (robot description, URDF)
Before this commit: robot frog, 45 links, 44 joints
Joints:
- joint LShank_ry: child LShank_rz -> LShank_ry
- joint LShank_rz: parent LShank_rz -> LShank_ry

File: data/urdf/spiderman/spiderman.urdf (robot description, URDF)
Before this commit: robot spiderman, 38 links, 37 joints
Joints:
- joint LFoot_rx: child LFoot_ry -> LFoot_rx
- joint RFoot_rz: parent RFoot_ry -> RFoot_rx
