Commit message: Remove antena DOF of Ant, update extending and flexion configs in scripts

File: data/urdf/ant/LBFootSphere.urdf (robot description, URDF)
Before this commit: robot LBFootSphere, 21 links, 20 joints
Links:
- removed link LAntenaFoot_rx
- removed link LAntenaFoot_ry
- removed link LAntena_rx
- removed link LAntena_ry
- removed link RAntenaFoot_rx
- removed link RAntenaFoot_ry
- removed link RAntena_rx
- removed link RAntena_ry
Joints:
- removed joint LAntenaFoot_rx
- removed joint LAntenaFoot_ry
- removed joint LAntenaFoot_rz
- removed joint LAntena_rx
- removed joint LAntena_ry
- removed joint LAntena_rz
- removed joint RAntenaFoot_rx
- removed joint RAntenaFoot_ry
- removed joint RAntenaFoot_rz
- removed joint RAntena_rx
- removed joint RAntena_ry
- removed joint RAntena_rz
- added joint LAntena: type fixed, parent Head, child LAntena, origin xyz=0.0176 -0.1027 0.0225 rpy=0 0 0
- added joint LAntenaFoot: type fixed, parent LAntena, child LAntenaFoot, origin xyz=0.0267 -0.0198 0.1006 rpy=0 0 0
- added joint RAntena: type fixed, parent Head, child RAntena, origin xyz=-0.0168 -0.1029 0.0226 rpy=0 0 0
- added joint RAntenaFoot: type fixed, parent RAntena, child RAntenaFoot, origin xyz=-0.0279 -0.0202 0.1006 rpy=0 0 0

File: data/urdf/ant/LFFootSphere.urdf (robot description, URDF)
Before this commit: robot LFFootSphere, 21 links, 20 joints
Links:
- removed link LAntenaFoot_rx
- removed link LAntenaFoot_ry
- removed link LAntena_rx
- removed link LAntena_ry
- removed link RAntenaFoot_rx
- removed link RAntenaFoot_ry
- removed link RAntena_rx
- removed link RAntena_ry
Joints:
- removed joint LAntenaFoot_rx
- removed joint LAntenaFoot_ry
- removed joint LAntenaFoot_rz
- removed joint LAntena_rx
- removed joint LAntena_ry
- removed joint LAntena_rz
- removed joint RAntenaFoot_rx
- removed joint RAntenaFoot_ry
- removed joint RAntenaFoot_rz
- removed joint RAntena_rx
- removed joint RAntena_ry
- removed joint RAntena_rz
- added joint LAntena: type fixed, parent Head, child LAntena, origin xyz=0.0176 -0.1027 0.0225 rpy=0 0 0
- added joint LAntenaFoot: type fixed, parent LAntena, child LAntenaFoot, origin xyz=0.0267 -0.0198 0.1006 rpy=0 0 0
- added joint RAntena: type fixed, parent Head, child RAntena, origin xyz=-0.0168 -0.1029 0.0226 rpy=0 0 0
- added joint RAntenaFoot: type fixed, parent RAntena, child RAntenaFoot, origin xyz=-0.0279 -0.0202 0.1006 rpy=0 0 0

File: data/urdf/ant/LMFootSphere.urdf (robot description, URDF)
Before this commit: robot LMFootSphere, 21 links, 20 joints
Links:
- removed link LAntenaFoot_rx
- removed link LAntenaFoot_ry
- removed link LAntena_rx
- removed link LAntena_ry
- removed link RAntenaFoot_rx
- removed link RAntenaFoot_ry
- removed link RAntena_rx
- removed link RAntena_ry
Joints:
- removed joint LAntenaFoot_rx
- removed joint LAntenaFoot_ry
- removed joint LAntenaFoot_rz
- removed joint LAntena_rx
- removed joint LAntena_ry
- removed joint LAntena_rz
- removed joint RAntenaFoot_rx
- removed joint RAntenaFoot_ry
- removed joint RAntenaFoot_rz
- removed joint RAntena_rx
- removed joint RAntena_ry
- removed joint RAntena_rz
- added joint LAntena: type fixed, parent Head, child LAntena, origin xyz=0.0176 -0.1027 0.0225 rpy=0 0 0
- added joint LAntenaFoot: type fixed, parent LAntena, child LAntenaFoot, origin xyz=0.0267 -0.0198 0.1006 rpy=0 0 0
- added joint RAntena: type fixed, parent Head, child RAntena, origin xyz=-0.0168 -0.1029 0.0226 rpy=0 0 0
- added joint RAntenaFoot: type fixed, parent RAntena, child RAntenaFoot, origin xyz=-0.0279 -0.0202 0.1006 rpy=0 0 0

File: data/urdf/ant/RBFootSphere.urdf (robot description, URDF)
Before this commit: robot RBFootSphere, 21 links, 20 joints
Links:
- removed link LAntenaFoot_rx
- removed link LAntenaFoot_ry
- removed link LAntena_rx
- removed link LAntena_ry
- removed link RAntenaFoot_rx
- removed link RAntenaFoot_ry
- removed link RAntena_rx
- removed link RAntena_ry
Joints:
- removed joint LAntenaFoot_rx
- removed joint LAntenaFoot_ry
- removed joint LAntenaFoot_rz
- removed joint LAntena_rx
- removed joint LAntena_ry
- removed joint LAntena_rz
- removed joint RAntenaFoot_rx
- removed joint RAntenaFoot_ry
- removed joint RAntenaFoot_rz
- removed joint RAntena_rx
- removed joint RAntena_ry
- removed joint RAntena_rz
- added joint LAntena: type fixed, parent Head, child LAntena, origin xyz=0.0176 -0.1027 0.0225 rpy=0 0 0
- added joint LAntenaFoot: type fixed, parent LAntena, child LAntenaFoot, origin xyz=0.0267 -0.0198 0.1006 rpy=0 0 0
- added joint RAntena: type fixed, parent Head, child RAntena, origin xyz=-0.0168 -0.1029 0.0226 rpy=0 0 0
- added joint RAntenaFoot: type fixed, parent RAntena, child RAntenaFoot, origin xyz=-0.0279 -0.0202 0.1006 rpy=0 0 0

File: data/urdf/ant/RFFootSphere.urdf (robot description, URDF)
Before this commit: robot RFFootSphere, 21 links, 20 joints
Links:
- removed link LAntenaFoot_rx
- removed link LAntenaFoot_ry
- removed link LAntena_rx
- removed link LAntena_ry
- removed link RAntenaFoot_rx
- removed link RAntenaFoot_ry
- removed link RAntena_rx
- removed link RAntena_ry
Joints:
- removed joint LAntenaFoot_rx
- removed joint LAntenaFoot_ry
- removed joint LAntenaFoot_rz
- removed joint LAntena_rx
- removed joint LAntena_ry
- removed joint LAntena_rz
- removed joint RAntenaFoot_rx
- removed joint RAntenaFoot_ry
- removed joint RAntenaFoot_rz
- removed joint RAntena_rx
- removed joint RAntena_ry
- removed joint RAntena_rz
- added joint LAntena: type fixed, parent Head, child LAntena, origin xyz=0.0176 -0.1027 0.0225 rpy=0 0 0
- added joint LAntenaFoot: type fixed, parent LAntena, child LAntenaFoot, origin xyz=0.0267 -0.0198 0.1006 rpy=0 0 0
- added joint RAntena: type fixed, parent Head, child RAntena, origin xyz=-0.0168 -0.1029 0.0226 rpy=0 0 0
- added joint RAntenaFoot: type fixed, parent RAntena, child RAntenaFoot, origin xyz=-0.0279 -0.0202 0.1006 rpy=0 0 0

File: data/urdf/ant/RMFootSphere.urdf (robot description, URDF)
Before this commit: robot RMFootSphere, 21 links, 20 joints
Links:
- removed link LAntenaFoot_rx
- removed link LAntenaFoot_ry
- removed link LAntena_rx
- removed link LAntena_ry
- removed link RAntenaFoot_rx
- removed link RAntenaFoot_ry
- removed link RAntena_rx
- removed link RAntena_ry
Joints:
- removed joint LAntenaFoot_rx
- removed joint LAntenaFoot_ry
- removed joint LAntenaFoot_rz
- removed joint LAntena_rx
- removed joint LAntena_ry
- removed joint LAntena_rz
- removed joint RAntenaFoot_rx
- removed joint RAntenaFoot_ry
- removed joint RAntenaFoot_rz
- removed joint RAntena_rx
- removed joint RAntena_ry
- removed joint RAntena_rz
- added joint LAntena: type fixed, parent Head, child LAntena, origin xyz=0.0176 -0.1027 0.0225 rpy=0 0 0
- added joint LAntenaFoot: type fixed, parent LAntena, child LAntenaFoot, origin xyz=0.0267 -0.0198 0.1006 rpy=0 0 0
- added joint RAntena: type fixed, parent Head, child RAntena, origin xyz=-0.0168 -0.1029 0.0226 rpy=0 0 0
- added joint RAntenaFoot: type fixed, parent RAntena, child RAntenaFoot, origin xyz=-0.0279 -0.0202 0.1006 rpy=0 0 0

File: data/urdf/ant/ant.urdf (robot description, URDF)
Before this commit: robot articulated_ant, 81 links, 80 joints
Links:
- removed link LAntenaFoot_rx
- removed link LAntenaFoot_ry
- removed link LAntena_rx
- removed link LAntena_ry
- removed link RAntenaFoot_rx
- removed link RAntenaFoot_ry
- removed link RAntena_rx
- removed link RAntena_ry
Joints:
- removed joint LAntenaFoot_rx
- removed joint LAntenaFoot_ry
- removed joint LAntenaFoot_rz
- removed joint LAntena_rx
- removed joint LAntena_ry
- removed joint LAntena_rz
- removed joint RAntenaFoot_rx
- removed joint RAntenaFoot_ry
- removed joint RAntenaFoot_rz
- removed joint RAntena_rx
- removed joint RAntena_ry
- removed joint RAntena_rz
- added joint LAntena: type fixed, parent Head, child LAntena, origin xyz=0.0176 -0.1027 0.0225 rpy=0 0 0
- added joint LAntenaFoot: type fixed, parent LAntena, child LAntenaFoot, origin xyz=0.0267 -0.0198 0.1006 rpy=0 0 0
- added joint RAntena: type fixed, parent Head, child RAntena, origin xyz=-0.0168 -0.1029 0.0226 rpy=0 0 0
- added joint RAntenaFoot: type fixed, parent RAntena, child RAntenaFoot, origin xyz=-0.0279 -0.0202 0.1006 rpy=0 0 0

File: data/urdf/ant/ant_trunk.urdf (robot description, URDF)
Before this commit: robot ant_trunk, 20 links, 19 joints
Links:
- removed link LAntenaFoot_rx
- removed link LAntenaFoot_ry
- removed link LAntena_rx
- removed link LAntena_ry
- removed link RAntenaFoot_rx
- removed link RAntenaFoot_ry
- removed link RAntena_rx
- removed link RAntena_ry
Joints:
- removed joint LAntenaFoot_rx
- removed joint LAntenaFoot_ry
- removed joint LAntenaFoot_rz
- removed joint LAntena_rx
- removed joint LAntena_ry
- removed joint LAntena_rz
- removed joint RAntenaFoot_rx
- removed joint RAntenaFoot_ry
- removed joint RAntenaFoot_rz
- removed joint RAntena_rx
- removed joint RAntena_ry
- removed joint RAntena_rz
- added joint LAntena: type fixed, parent Head, child LAntena, origin xyz=0.0176 -0.1027 0.0225 rpy=0 0 0
- added joint LAntenaFoot: type fixed, parent LAntena, child LAntenaFoot, origin xyz=0.0267 -0.0198 0.1006 rpy=0 0 0
- added joint RAntena: type fixed, parent Head, child RAntena, origin xyz=-0.0168 -0.1029 0.0226 rpy=0 0 0
- added joint RAntenaFoot: type fixed, parent RAntena, child RAntenaFoot, origin xyz=-0.0279 -0.0202 0.1006 rpy=0 0 0

Commit message: Remove offset in ant thorax, adapt armature, ROMs, URDF... Ant skinning now working

File: data/urdf/ant/LBFootSphere.urdf (robot description, URDF)
Before this commit: robot LBFootSphere, 13 links, 12 joints
Joints:
- joint Abdomen_rx: origin xyz=0 0.15853 0.19806 rpy=0 0 0 -> xyz=0 0.1203 -0.0006 rpy=0 0 0
- joint Head_rx: origin xyz=0 -0.06471 0.21279 rpy=0 0 0 -> xyz=0 -0.1029 0.0142 rpy=0 0 0
- joint base_link_J: origin xyz=0.001 -0.0382 -0.1982 rpy=0 0 1.570796 -> xyz=0 0 0 rpy=0 0 1.570796

File: data/urdf/ant/LFFootSphere.urdf (robot description, URDF)
Before this commit: robot LFFootSphere, 13 links, 12 joints
Joints:
- joint Abdomen_rx: origin xyz=0 0.15853 0.19806 rpy=0 0 0 -> xyz=0 0.1203 -0.0006 rpy=0 0 0
- joint Head_rx: origin xyz=0 -0.06471 0.21279 rpy=0 0 0 -> xyz=0 -0.1029 0.0142 rpy=0 0 0
- joint base_link_J: origin xyz=0.001 -0.0382 -0.1982 rpy=0 0 1.570796 -> xyz=0 0 0 rpy=0 0 1.570796

File: data/urdf/ant/LMFootSphere.urdf (robot description, URDF)
Before this commit: robot LMFootSphere, 13 links, 12 joints
Joints:
- joint Abdomen_rx: origin xyz=0 0.15853 0.19806 rpy=0 0 0 -> xyz=0 0.1203 -0.0006 rpy=0 0 0
- joint Head_rx: origin xyz=0 -0.06471 0.21279 rpy=0 0 0 -> xyz=0 -0.1029 0.0142 rpy=0 0 0
- joint base_link_J: origin xyz=0.001 -0.0382 -0.1982 rpy=0 0 1.570796 -> xyz=0 0 0 rpy=0 0 1.570796

File: data/urdf/ant/RBFootSphere.urdf (robot description, URDF)
Before this commit: robot RBFootSphere, 13 links, 12 joints
Joints:
- joint Abdomen_rx: origin xyz=0 0.15853 0.19806 rpy=0 0 0 -> xyz=0 0.1203 -0.0006 rpy=0 0 0
- joint Head_rx: origin xyz=0 -0.06471 0.21279 rpy=0 0 0 -> xyz=0 -0.1029 0.0142 rpy=0 0 0
- joint base_link_J: origin xyz=0.001 -0.0382 -0.1982 rpy=0 0 1.570796 -> xyz=0 0 0 rpy=0 0 1.570796

File: data/urdf/ant/RFFootSphere.urdf (robot description, URDF)
Before this commit: robot RFFootSphere, 13 links, 12 joints
Joints:
- joint Abdomen_rx: origin xyz=0 0.15853 0.19806 rpy=0 0 0 -> xyz=0 0.1203 -0.0006 rpy=0 0 0
- joint Head_rx: origin xyz=0 -0.06471 0.21279 rpy=0 0 0 -> xyz=0 -0.1029 0.0142 rpy=0 0 0
- joint base_link_J: origin xyz=0.001 -0.0382 -0.1982 rpy=0 0 1.570796 -> xyz=0 0 0 rpy=0 0 1.570796

File: data/urdf/ant/RMFootSphere.urdf (robot description, URDF)
Before this commit: robot RMFootSphere, 13 links, 12 joints
Joints:
- joint Abdomen_rx: origin xyz=0 0.15853 0.19806 rpy=0 0 0 -> xyz=0 0.1203 -0.0006 rpy=0 0 0
- joint Head_rx: origin xyz=0 -0.06471 0.21279 rpy=0 0 0 -> xyz=0 -0.1029 0.0142 rpy=0 0 0
- joint base_link_J: origin xyz=0.001 -0.0382 -0.1982 rpy=0 0 1.570796 -> xyz=0 0 0 rpy=0 0 1.570796

File: data/urdf/ant/ant.urdf (robot description, URDF)
Before this commit: robot articulated_ant, 73 links, 72 joints
Joints:
- joint Abdomen_rx: origin xyz=0 0.15853 0.19806 rpy=0 0 0 -> xyz=0 0.1203 -0.0006 rpy=0 0 0
- joint Head_rx: origin xyz=0 -0.06471 0.21279 rpy=0 0 0 -> xyz=0 -0.1029 0.0142 rpy=0 0 0
- joint LBThigh_rx: origin xyz=0.06238 0.08879 0.18588 rpy=0 0 0 -> xyz=0.0624 0.0506 -0.0127 rpy=0 0 0
- joint LFThigh_rx: origin xyz=0.0743 -0.0223 0.1894 rpy=0 0 0 -> xyz=0.0743 -0.0605 -0.0092 rpy=0 0 0
- joint LMThigh_rx: origin xyz=0.07469 0.03933 0.19123 rpy=0 0 0 -> xyz=0.0747 0.0011 -0.0074 rpy=0 0 0
- joint RBThigh_rx: origin xyz=-0.06230 0.08906 0.18543 rpy=0 0 0 -> xyz=-0.0623 0.0509 -0.0132 rpy=0 0 0
- joint RFThigh_rx: origin xyz=-0.07030 -0.02046 0.18987 rpy=0 0 0 -> xyz=-0.0703 -0.0587 -0.0088 rpy=0 0 0
- joint RMThigh_rx: origin xyz=-0.07457 0.03980 0.19130 rpy=0 0 0 -> xyz=-0.0746 0.0016 -0.0073 rpy=0 0 0
- joint base_link_J: origin xyz=0.001 -0.0382 -0.1982 rpy=0 0 1.570796 -> xyz=0 0 0 rpy=0 0 1.570796

File: data/urdf/ant/ant_trunk.urdf (robot description, URDF)
Before this commit: robot ant_trunk, 12 links, 11 joints
Joints:
- joint Abdomen_rx: origin xyz=0 0.15853 0.19806 rpy=0 0 0 -> xyz=0 0.1203 -0.0006 rpy=0 0 0
- joint Head_rx: origin xyz=0 -0.06471 0.21279 rpy=0 0 0 -> xyz=0 -0.1029 0.0142 rpy=0 0 0
- joint base_link_J: origin xyz=0.001 -0.0382 -0.1982 rpy=0 0 1.570796 -> xyz=0 0 0 rpy=0 0 1.570796

Commit message: Update ant scripts for COM, add COM-shift in URDF

File: data/urdf/ant/LBFootSphere.urdf (robot description, URDF)
Before this commit: robot LBFootSphere, 13 links, 12 joints
Links:
- added link base_link_comshift
Joints:
- added joint base_link_comshift_J: type fixed, parent base_link_comshift, child Thorax, origin xyz=0 -0.01066 -0.003041 rpy=0 0 0
- joint base_link_J: child Thorax -> base_link_comshift

File: data/urdf/ant/LFFootSphere.urdf (robot description, URDF)
Before this commit: robot LFFootSphere, 13 links, 12 joints
Links:
- added link base_link_comshift
Joints:
- added joint base_link_comshift_J: type fixed, parent base_link_comshift, child Thorax, origin xyz=0 -0.01066 -0.003041 rpy=0 0 0
- joint base_link_J: child Thorax -> base_link_comshift

File: data/urdf/ant/LMFootSphere.urdf (robot description, URDF)
Before this commit: robot LMFootSphere, 13 links, 12 joints
Links:
- added link base_link_comshift
Joints:
- added joint base_link_comshift_J: type fixed, parent base_link_comshift, child Thorax, origin xyz=0 -0.01066 -0.003041 rpy=0 0 0
- joint base_link_J: child Thorax -> base_link_comshift

File: data/urdf/ant/RBFootSphere.urdf (robot description, URDF)
Before this commit: robot RBFootSphere, 13 links, 12 joints
Links:
- added link base_link_comshift
Joints:
- added joint base_link_comshift_J: type fixed, parent base_link_comshift, child Thorax, origin xyz=0 -0.01066 -0.003041 rpy=0 0 0
- joint base_link_J: child Thorax -> base_link_comshift

File: data/urdf/ant/RFFootSphere.urdf (robot description, URDF)
Before this commit: robot RFFootSphere, 13 links, 12 joints
Links:
- added link base_link_comshift
Joints:
- added joint base_link_comshift_J: type fixed, parent base_link_comshift, child Thorax, origin xyz=0 -0.01066 -0.003041 rpy=0 0 0
- joint base_link_J: child Thorax -> base_link_comshift

File: data/urdf/ant/RMFootSphere.urdf (robot description, URDF)
Before this commit: robot RMFootSphere, 13 links, 12 joints
Links:
- added link base_link_comshift
Joints:
- added joint base_link_comshift_J: type fixed, parent base_link_comshift, child Thorax, origin xyz=0 -0.01066 -0.003041 rpy=0 0 0
- joint base_link_J: child Thorax -> base_link_comshift

File: data/urdf/ant/ant.urdf (robot description, URDF)
Before this commit: robot articulated_ant, 73 links, 72 joints
Links:
- added link base_link_comshift
- link Abdomen: mass 1.5 -> 5
- link Head: mass 1.3 -> 5
- link LAntena: mass 0.05 -> 0
- link LAntenaFoot: mass 0.05 -> 0
- link LBFoot: mass 0.1 -> 0.4
- link LBShank: mass 0.2 -> 0.5
- link LBThigh: mass 0.3 -> 0.6
- link LFFoot: mass 0.1 -> 0.4
- link LFShank: mass 0.2 -> 0.5
- link LFThigh: mass 0.3 -> 0.6
- link LMFoot: mass 0.1 -> 0.4
- link LMShank: mass 0.2 -> 0.5
- link LMThigh: mass 0.3 -> 0.6
- link RAntena: mass 0.05 -> 0
- link RAntenaFoot: mass 0.05 -> 0
- link RBFoot: mass 0.1 -> 0.4
- link RBShank: mass 0.2 -> 0.5
- link RBThigh: mass 0.3 -> 0.6
- link RFFoot: mass 0.1 -> 0.4
- link RFShank: mass 0.2 -> 0.5
- link RFThigh: mass 0.3 -> 0.6
- link RMFoot: mass 0.1 -> 0.4
- link RMShank: mass 0.2 -> 0.5
- link RMThigh: mass 0.3 -> 0.6
- link Thorax: mass 2 -> 6
Joints:
- added joint base_link_comshift_J: type fixed, parent base_link_comshift, child Thorax, origin xyz=0 -0.01066 -0.003041 rpy=0 0 0
- joint base_link_J: child Thorax -> base_link_comshift
- joint virtualThorax: parent base_link -> Thorax

File: data/urdf/ant/ant_trunk.urdf (robot description, URDF)
Before this commit: robot ant_trunk, 12 links, 11 joints
Links:
- added link base_link_comshift
- link LAntena: mass 1 -> None; geometry 
- link LAntenaFoot: mass 1 -> None; geometry 
- link RAntena: mass 1 -> None; geometry 
- link RAntenaFoot: mass 1 -> None; geometry 
Joints:
- added joint base_link_comshift_J: type fixed, parent base_link_comshift, child Thorax, origin xyz=0 -0.01066 -0.003041 rpy=0 0 0
- joint base_link_J: child Thorax -> base_link_comshift
