Commit message: Lamp: fix trunk (for contact creation), add plateform waypoints, update scripts

File: data/urdf/lamp/lamp_trunk.urdf (robot description, URDF)
Before this commit: robot lamp_trunk, 4 links, 3 joints
Links:
- added link head_rom; visual mesh filename=package://hpp-rbprm-corba/meshes/lamp/foot_rom.stl
- link Head: geometry collision mesh filename=package://hpp-rbprm-corba/meshes/lamp/Head_box.stl; visual mesh filename=package://hpp-rbprm-corba/meshes/lamp/Head_box.stl
Joints:
- added joint head_rom_joint: type fixed, parent HeadLink, child head_rom, origin xyz=0 0 0 rpy=0 0 0
