Commit message: Add 1 DOF to jumping-lamp

File: data/urdf/lamp/lamp.urdf (robot description, URDF)
Before this commit: robot lamp, 12 links, 11 joints
Links:
- added link ThighJointBis
- added link head_rom; visual mesh filename=package://hpp-rbprm-corba/meshes/lamp/foot_rom.stl
Joints:
- added joint ThighJointBis: type revolute, parent ThighJoint, child ThighJointBis, origin xyz=0 0 0 rpy=0 0 0, axis 0 1 0, limit lower=-0.55 upper=0.05 effort=0 velocity=1.0
- added joint head_rom_joint: type fixed, parent HeadLink, child head_rom, origin xyz=0 0 0 rpy=0 0 0
- joint Thigh: parent ThighJoint -> ThighJointBis

Commit message: Transition to constrained comRRT (not finished):
- add function to get lastStatesComputedTime stack
- update lastStatesComputedTime with ballistic-interpolation, PATH RETURNING IS COMMITED
- set new refConfigs in Skeleton scripts
- set realistic mass values for Lamp (for CoM)

File: data/urdf/lamp/lamp.urdf (robot description, URDF)
Before this commit: robot lamp, 14 links, 13 joints
Links:
- link Ankle: mass 1 -> 0.08
- link Foot: mass 1 -> 1.
- link Head: mass 1 -> 2.8
- link Shank: mass 1 -> 0.5
- link Thigh: mass 1 -> 0.5

Commit message: Increase lamp joint limits, FIX lamp ROM

File: data/urdf/lamp/lamp.urdf (robot description, URDF)
Before this commit: robot lamp, 14 links, 13 joints
Joints:
- joint LampFootSphere: origin xyz=0 0 -0.007 rpy=0 0 0 -> xyz=0 0 -0.007 rpy=0 0 3.1415926535
- joint ShankJoint: limit lower=-2.6 upper=2.1 effort=0 velocity=1.0 -> lower=-2.8 upper=2.1 effort=0 velocity=1.0
- joint ThighJointBis: limit lower=-0.55 upper=0.05 effort=0 velocity=1.0 -> lower=-1.2 upper=0.25 effort=0 velocity=1.0

File: data/urdf/lamp/lamp_trunk.urdf (robot description, URDF)
Before this commit: robot lamp_trunk, 3 links, 2 joints
Links:
- added link base_link_comshift
- added link head_rom; visual mesh filename=package://hpp-rbprm-corba/meshes/lamp/foot_rom.stl
Joints:
- added joint base_link_comshift_J: type fixed, parent base_link_comshift, child Head, origin xyz=-0.023 0 0.245 rpy=0 0 0
- added joint head_rom_joint: type fixed, parent HeadLink, child head_rom, origin xyz=0 0 0 rpy=0 0 0
- joint base_link_J: child Head -> base_link_comshift

Commit message: Fix lamp ROM in head_view, add head_box

File: data/urdf/lamp/lamp.urdf (robot description, URDF)
Before this commit: robot lamp, 14 links, 13 joints
Links:
- added link head_rom; visual mesh filename=package://hpp-rbprm-corba/meshes/lamp/foot_rom.stl
Joints:
- added joint head_rom_joint: type fixed, parent HeadLink, child head_rom, origin xyz=0 0 0 rpy=0 0 0

File: data/urdf/lamp/lamp_trunk.urdf (robot description, URDF)
Before this commit: robot lamp_trunk, 5 links, 4 joints
Links:
- link Head: geometry collision mesh filename=package://hpp-rbprm-corba/meshes/lamp/Head_box.stl; visual mesh filename=package://hpp-rbprm-corba/meshes/lamp/Head_view.dae
- link HeadLink: geometry visual mesh filename=package://hpp-rbprm-corba/meshes/lamp/HeadLink.stl

Commit message: Add Lamp masses, fix blender

File: data/urdf/lamp/lamp.urdf (robot description, URDF)
Before this commit: robot lamp, 14 links, 13 joints
Links:
- link Ankle: mass 0.08 -> 0.8
- link Foot: mass 1. -> 10
- link Head: mass 2.8 -> 28
- link Shank: mass 0.5 -> 5
- link Thigh: mass 0.5 -> 5
