Commit message: Add cone models, resize skeleton ROMs, change parkourWalls

File: data/urdf/skeleton/skeleton_trunk.urdf (robot description, URDF)
Before this commit: robot skeleton_trunk_flexible, 26 links, 25 joints
Links:
- added link ThoraxShift
- added link pelvis_lfoot_rom; visual mesh filename=package://hpp-rbprm-corba/meshes/skeleton/lfoot_rom.stl
- added link pelvis_rfoot_rom; visual mesh filename=package://hpp-rbprm-corba/meshes/skeleton/rfoot_rom.stl
- added link thorax_lhand_rom; visual mesh filename=package://hpp-rbprm-corba/meshes/skeleton/lhand_rom.stl
- added link thorax_rhand_rom; visual mesh filename=package://hpp-rbprm-corba/meshes/skeleton/rhand_rom.stl
- link Pelvis: geometry collision mesh filename=package://hpp-rbprm-corba/meshes/skeleton/pelvis_box.stl; visual mesh filename=package://hpp-rbprm-corba/meshes/skeleton/pelvis_box.stl
- link Skull: geometry collision mesh filename=package://hpp-rbprm-corba/meshes/skeleton/skull_box.stl; visual mesh filename=package://hpp-rbprm-corba/meshes/skeleton/skull_box.stl
- link Thorax: geometry collision mesh filename=package://hpp-rbprm-corba/meshes/skeleton/thorax_box.stl; visual mesh filename=package://hpp-rbprm-corba/meshes/skeleton/thorax_box.stl
Joints:
- added joint ThoraxShift: type fixed, parent ThoraxShift, child Thorax, origin xyz=0.035889 0 0.14072 rpy=0 0 0
- added joint pelvis_lfoot_rom_joint: type fixed, parent Pelvis, child pelvis_lfoot_rom, origin xyz=0 0 0 rpy=0 0 0
- added joint pelvis_rfoot_rom_joint: type fixed, parent Pelvis, child pelvis_rfoot_rom, origin xyz=0 0 0 rpy=0 0 0
- added joint thorax_lhand_rom_joint: type fixed, parent ThoraxShift, child thorax_lhand_rom, origin xyz=0 0 0 rpy=0 0 0
- added joint thorax_rhand_rom_joint: type fixed, parent ThoraxShift, child thorax_rhand_rom, origin xyz=0 0 0 rpy=0 0 0
- joint A_ThoraxSkull_J1: parent Thorax -> ThoraxShift
- joint Thorax: child Thorax -> ThoraxShift
