Commit message: Remove spine-DOF of skeleton

File: data/urdf/skeleton/LFootSphere.urdf (robot description, URDF)
Before this commit: robot LFootSphere, 27 links, 26 joints
Links:
- added link ThoraxShift
Joints:
- added joint ThoraxShift: type fixed, parent ThoraxShift, child Thorax, origin xyz=0.035889 0 0.14072 rpy=0 0 0
- joint L1: axis 0 1 0 -> (none); limit lower=-0.1 upper=0.1 effort=0 velocity=1.0 -> (none); type revolute -> fixed
- joint L1Thorax_J1: limit lower=-0.2 upper=0.2 effort=0 velocity=1.0 -> lower=-0.3 upper=0.3 effort=0 velocity=1.0
- joint L2: axis 0 1 0 -> (none); limit lower=-0.1 upper=0.1 effort=0 velocity=1.0 -> (none); type revolute -> fixed
- joint L2L1_J1: axis 1 0 0 -> (none); limit lower=-0.1 upper=0.1 effort=0 velocity=1.0 -> (none); type revolute -> fixed
- joint L2L1_J2: axis 0 0 1 -> (none); limit lower=-0.1 upper=0.1 effort=0 velocity=1.0 -> (none); type revolute -> fixed
- joint L3: axis 0 1 0 -> (none); limit lower=-0.1 upper=0.1 effort=0 velocity=1.0 -> (none); type revolute -> fixed
- joint L3L2_J1: axis 1 0 0 -> (none); limit lower=-0.1 upper=0.1 effort=0 velocity=1.0 -> (none); type revolute -> fixed
- joint L3L2_J2: axis 0 0 1 -> (none); limit lower=-0.1 upper=0.1 effort=0 velocity=1.0 -> (none); type revolute -> fixed
- joint L4: axis 0 1 0 -> (none); limit lower=-0.1 upper=0.1 effort=0 velocity=1.0 -> (none); type revolute -> fixed
- joint L4L3_J1: axis 1 0 0 -> (none); limit lower=-0.1 upper=0.1 effort=0 velocity=1.0 -> (none); type revolute -> fixed
- joint L4L3_J2: axis 0 0 1 -> (none); limit lower=-0.1 upper=0.1 effort=0 velocity=1.0 -> (none); type revolute -> fixed
- joint L5: axis 0 1 0 -> (none); limit lower=-0.1 upper=0.1 effort=0 velocity=1.0 -> (none); type revolute -> fixed
- joint L5L4_J1: axis 1 0 0 -> (none); limit lower=-0.1 upper=0.1 effort=0 velocity=1.0 -> (none); type revolute -> fixed
- joint L5L4_J2: axis 0 0 1 -> (none); limit lower=-0.1 upper=0.1 effort=0 velocity=1.0 -> (none); type revolute -> fixed
- joint SacrumL5_J1: axis 1 0 0 -> (none); limit lower=-0.1 upper=0.1 effort=0 velocity=1.0 -> (none); type revolute -> fixed
- joint SacrumL5_J2: axis 0 0 1 -> (none); limit lower=-0.1 upper=0.1 effort=0 velocity=1.0 -> (none); type revolute -> fixed
- joint Thorax: child Thorax -> ThoraxShift; limit lower=-0.5 upper=0.6 effort=0 velocity=1.0 -> lower=-0.6 upper=0.7 effort=0 velocity=1.0

File: data/urdf/skeleton/LHandSphere.urdf (robot description, URDF)
Before this commit: robot LHandSphere, 27 links, 26 joints
Links:
- added link ThoraxShift
Joints:
- added joint ThoraxShift: type fixed, parent ThoraxShift, child Thorax, origin xyz=0.035889 0 0.14072 rpy=0 0 0
- joint L1: axis 0 1 0 -> (none); limit lower=-0.1 upper=0.1 effort=0 velocity=1.0 -> (none); type revolute -> fixed
- joint L1Thorax_J1: limit lower=-0.2 upper=0.2 effort=0 velocity=1.0 -> lower=-0.3 upper=0.3 effort=0 velocity=1.0
- joint L2: axis 0 1 0 -> (none); limit lower=-0.1 upper=0.1 effort=0 velocity=1.0 -> (none); type revolute -> fixed
- joint L2L1_J1: axis 1 0 0 -> (none); limit lower=-0.1 upper=0.1 effort=0 velocity=1.0 -> (none); type revolute -> fixed
- joint L2L1_J2: axis 0 0 1 -> (none); limit lower=-0.1 upper=0.1 effort=0 velocity=1.0 -> (none); type revolute -> fixed
- joint L3: axis 0 1 0 -> (none); limit lower=-0.1 upper=0.1 effort=0 velocity=1.0 -> (none); type revolute -> fixed
- joint L3L2_J1: axis 1 0 0 -> (none); limit lower=-0.1 upper=0.1 effort=0 velocity=1.0 -> (none); type revolute -> fixed
- joint L3L2_J2: axis 0 0 1 -> (none); limit lower=-0.1 upper=0.1 effort=0 velocity=1.0 -> (none); type revolute -> fixed
- joint L4: axis 0 1 0 -> (none); limit lower=-0.1 upper=0.1 effort=0 velocity=1.0 -> (none); type revolute -> fixed
- joint L4L3_J1: axis 1 0 0 -> (none); limit lower=-0.1 upper=0.1 effort=0 velocity=1.0 -> (none); type revolute -> fixed
- joint L4L3_J2: axis 0 0 1 -> (none); limit lower=-0.1 upper=0.1 effort=0 velocity=1.0 -> (none); type revolute -> fixed
- joint L5: axis 0 1 0 -> (none); limit lower=-0.1 upper=0.1 effort=0 velocity=1.0 -> (none); type revolute -> fixed
- joint L5L4_J1: axis 1 0 0 -> (none); limit lower=-0.1 upper=0.1 effort=0 velocity=1.0 -> (none); type revolute -> fixed
- joint L5L4_J2: axis 0 0 1 -> (none); limit lower=-0.1 upper=0.1 effort=0 velocity=1.0 -> (none); type revolute -> fixed
- joint SacrumL5_J1: axis 1 0 0 -> (none); limit lower=-0.1 upper=0.1 effort=0 velocity=1.0 -> (none); type revolute -> fixed
- joint SacrumL5_J2: axis 0 0 1 -> (none); limit lower=-0.1 upper=0.1 effort=0 velocity=1.0 -> (none); type revolute -> fixed
- joint Thorax: child Thorax -> ThoraxShift; limit lower=-0.5 upper=0.6 effort=0 velocity=1.0 -> lower=-0.6 upper=0.7 effort=0 velocity=1.0

File: data/urdf/skeleton/RFootSphere.urdf (robot description, URDF)
Before this commit: robot RFootSphere, 27 links, 26 joints
Links:
- added link ThoraxShift
Joints:
- added joint ThoraxShift: type fixed, parent ThoraxShift, child Thorax, origin xyz=0.035889 0 0.14072 rpy=0 0 0
- joint L1: axis 0 1 0 -> (none); limit lower=-0.1 upper=0.1 effort=0 velocity=1.0 -> (none); type revolute -> fixed
- joint L1Thorax_J1: limit lower=-0.2 upper=0.2 effort=0 velocity=1.0 -> lower=-0.3 upper=0.3 effort=0 velocity=1.0
- joint L2: axis 0 1 0 -> (none); limit lower=-0.1 upper=0.1 effort=0 velocity=1.0 -> (none); type revolute -> fixed
- joint L2L1_J1: axis 1 0 0 -> (none); limit lower=-0.1 upper=0.1 effort=0 velocity=1.0 -> (none); type revolute -> fixed
- joint L2L1_J2: axis 0 0 1 -> (none); limit lower=-0.1 upper=0.1 effort=0 velocity=1.0 -> (none); type revolute -> fixed
- joint L3: axis 0 1 0 -> (none); limit lower=-0.1 upper=0.1 effort=0 velocity=1.0 -> (none); type revolute -> fixed
- joint L3L2_J1: axis 1 0 0 -> (none); limit lower=-0.1 upper=0.1 effort=0 velocity=1.0 -> (none); type revolute -> fixed
- joint L3L2_J2: axis 0 0 1 -> (none); limit lower=-0.1 upper=0.1 effort=0 velocity=1.0 -> (none); type revolute -> fixed
- joint L4: axis 0 1 0 -> (none); limit lower=-0.1 upper=0.1 effort=0 velocity=1.0 -> (none); type revolute -> fixed
- joint L4L3_J1: axis 1 0 0 -> (none); limit lower=-0.1 upper=0.1 effort=0 velocity=1.0 -> (none); type revolute -> fixed
- joint L4L3_J2: axis 0 0 1 -> (none); limit lower=-0.1 upper=0.1 effort=0 velocity=1.0 -> (none); type revolute -> fixed
- joint L5: axis 0 1 0 -> (none); limit lower=-0.1 upper=0.1 effort=0 velocity=1.0 -> (none); type revolute -> fixed
- joint L5L4_J1: axis 1 0 0 -> (none); limit lower=-0.1 upper=0.1 effort=0 velocity=1.0 -> (none); type revolute -> fixed
- joint L5L4_J2: axis 0 0 1 -> (none); limit lower=-0.1 upper=0.1 effort=0 velocity=1.0 -> (none); type revolute -> fixed
- joint SacrumL5_J1: axis 1 0 0 -> (none); limit lower=-0.1 upper=0.1 effort=0 velocity=1.0 -> (none); type revolute -> fixed
- joint SacrumL5_J2: axis 0 0 1 -> (none); limit lower=-0.1 upper=0.1 effort=0 velocity=1.0 -> (none); type revolute -> fixed
- joint Thorax: child Thorax -> ThoraxShift; limit lower=-0.5 upper=0.6 effort=0 velocity=1.0 -> lower=-0.6 upper=0.7 effort=0 velocity=1.0

File: data/urdf/skeleton/RHandSphere.urdf (robot description, URDF)
Before this commit: robot RHandSphere, 27 links, 26 joints
Links:
- added link ThoraxShift
Joints:
- added joint ThoraxShift: type fixed, parent ThoraxShift, child Thorax, origin xyz=0.035889 0 0.14072 rpy=0 0 0
- joint L1: axis 0 1 0 -> (none); limit lower=-0.1 upper=0.1 effort=0 velocity=1.0 -> (none); type revolute -> fixed
- joint L1Thorax_J1: limit lower=-0.2 upper=0.2 effort=0 velocity=1.0 -> lower=-0.3 upper=0.3 effort=0 velocity=1.0
- joint L2: axis 0 1 0 -> (none); limit lower=-0.1 upper=0.1 effort=0 velocity=1.0 -> (none); type revolute -> fixed
- joint L2L1_J1: axis 1 0 0 -> (none); limit lower=-0.1 upper=0.1 effort=0 velocity=1.0 -> (none); type revolute -> fixed
- joint L2L1_J2: axis 0 0 1 -> (none); limit lower=-0.1 upper=0.1 effort=0 velocity=1.0 -> (none); type revolute -> fixed
- joint L3: axis 0 1 0 -> (none); limit lower=-0.1 upper=0.1 effort=0 velocity=1.0 -> (none); type revolute -> fixed
- joint L3L2_J1: axis 1 0 0 -> (none); limit lower=-0.1 upper=0.1 effort=0 velocity=1.0 -> (none); type revolute -> fixed
- joint L3L2_J2: axis 0 0 1 -> (none); limit lower=-0.1 upper=0.1 effort=0 velocity=1.0 -> (none); type revolute -> fixed
- joint L4: axis 0 1 0 -> (none); limit lower=-0.1 upper=0.1 effort=0 velocity=1.0 -> (none); type revolute -> fixed
- joint L4L3_J1: axis 1 0 0 -> (none); limit lower=-0.1 upper=0.1 effort=0 velocity=1.0 -> (none); type revolute -> fixed
- joint L4L3_J2: axis 0 0 1 -> (none); limit lower=-0.1 upper=0.1 effort=0 velocity=1.0 -> (none); type revolute -> fixed
- joint L5: axis 0 1 0 -> (none); limit lower=-0.1 upper=0.1 effort=0 velocity=1.0 -> (none); type revolute -> fixed
- joint L5L4_J1: axis 1 0 0 -> (none); limit lower=-0.1 upper=0.1 effort=0 velocity=1.0 -> (none); type revolute -> fixed
- joint L5L4_J2: axis 0 0 1 -> (none); limit lower=-0.1 upper=0.1 effort=0 velocity=1.0 -> (none); type revolute -> fixed
- joint SacrumL5_J1: axis 1 0 0 -> (none); limit lower=-0.1 upper=0.1 effort=0 velocity=1.0 -> (none); type revolute -> fixed
- joint SacrumL5_J2: axis 0 0 1 -> (none); limit lower=-0.1 upper=0.1 effort=0 velocity=1.0 -> (none); type revolute -> fixed
- joint Thorax: child Thorax -> ThoraxShift; limit lower=-0.5 upper=0.6 effort=0 velocity=1.0 -> lower=-0.6 upper=0.7 effort=0 velocity=1.0

File: data/urdf/skeleton/armlessSkeleton_trunk.urdf (robot description, URDF)
Before this commit: robot armlessSkeleton_trunk, 26 links, 25 joints
Joints:
- joint L1: axis 0 1 0 -> (none); limit lower=-0.1 upper=0.1 effort=0 velocity=1.0 -> (none); type revolute -> fixed
- joint L1Thorax_J1: limit lower=-0.2 upper=0.2 effort=0 velocity=1.0 -> lower=-0.3 upper=0.3 effort=0 velocity=1.0
- joint L2: axis 0 1 0 -> (none); limit lower=-0.1 upper=0.1 effort=0 velocity=1.0 -> (none); type revolute -> fixed
- joint L2L1_J1: axis 1 0 0 -> (none); limit lower=-0.1 upper=0.1 effort=0 velocity=1.0 -> (none); type revolute -> fixed
- joint L2L1_J2: axis 0 0 1 -> (none); limit lower=-0.1 upper=0.1 effort=0 velocity=1.0 -> (none); type revolute -> fixed
- joint L3: axis 0 1 0 -> (none); limit lower=-0.1 upper=0.1 effort=0 velocity=1.0 -> (none); type revolute -> fixed
- joint L3L2_J1: axis 1 0 0 -> (none); limit lower=-0.1 upper=0.1 effort=0 velocity=1.0 -> (none); type revolute -> fixed
- joint L3L2_J2: axis 0 0 1 -> (none); limit lower=-0.1 upper=0.1 effort=0 velocity=1.0 -> (none); type revolute -> fixed
- joint L4: axis 0 1 0 -> (none); limit lower=-0.1 upper=0.1 effort=0 velocity=1.0 -> (none); type revolute -> fixed
- joint L4L3_J1: axis 1 0 0 -> (none); limit lower=-0.1 upper=0.1 effort=0 velocity=1.0 -> (none); type revolute -> fixed
- joint L4L3_J2: axis 0 0 1 -> (none); limit lower=-0.1 upper=0.1 effort=0 velocity=1.0 -> (none); type revolute -> fixed
- joint L5: axis 0 1 0 -> (none); limit lower=-0.1 upper=0.1 effort=0 velocity=1.0 -> (none); type revolute -> fixed
- joint L5L4_J1: axis 1 0 0 -> (none); limit lower=-0.1 upper=0.1 effort=0 velocity=1.0 -> (none); type revolute -> fixed
- joint L5L4_J2: axis 0 0 1 -> (none); limit lower=-0.1 upper=0.1 effort=0 velocity=1.0 -> (none); type revolute -> fixed
- joint SacrumL5_J1: axis 1 0 0 -> (none); limit lower=-0.1 upper=0.1 effort=0 velocity=1.0 -> (none); type revolute -> fixed
- joint SacrumL5_J2: axis 0 0 1 -> (none); limit lower=-0.1 upper=0.1 effort=0 velocity=1.0 -> (none); type revolute -> fixed
- joint Thorax: limit lower=-0.5 upper=0.6 effort=0 velocity=1.0 -> lower=-0.6 upper=0.7 effort=0 velocity=1.0

File: data/urdf/skeleton/skeleton.urdf (robot description, URDF)
Before this commit: robot skeleton, 58 links, 57 joints
Links:
- link LFoot: mass 0.72029 -> 0.52
- link RFoot: mass 0.72029 -> 0.52
Joints:
- joint L1: axis 0 1 0 -> (none); limit lower=-0.1 upper=0.1 effort=0 velocity=1.0 -> (none); type revolute -> fixed
- joint L1Thorax_J1: limit lower=-0.2 upper=0.2 effort=0 velocity=1.0 -> lower=-0.3 upper=0.3 effort=0 velocity=1.0
- joint L2: axis 0 1 0 -> (none); limit lower=-0.1 upper=0.1 effort=0 velocity=1.0 -> (none); type revolute -> fixed
- joint L2L1_J1: axis 1 0 0 -> (none); limit lower=-0.1 upper=0.1 effort=0 velocity=1.0 -> (none); type revolute -> fixed
- joint L2L1_J2: axis 0 0 1 -> (none); limit lower=-0.1 upper=0.1 effort=0 velocity=1.0 -> (none); type revolute -> fixed
- joint L3: axis 0 1 0 -> (none); limit lower=-0.1 upper=0.1 effort=0 velocity=1.0 -> (none); type revolute -> fixed
- joint L3L2_J1: axis 1 0 0 -> (none); limit lower=-0.1 upper=0.1 effort=0 velocity=1.0 -> (none); type revolute -> fixed
- joint L3L2_J2: axis 0 0 1 -> (none); limit lower=-0.1 upper=0.1 effort=0 velocity=1.0 -> (none); type revolute -> fixed
- joint L4: axis 0 1 0 -> (none); limit lower=-0.1 upper=0.1 effort=0 velocity=1.0 -> (none); type revolute -> fixed
- joint L4L3_J1: axis 1 0 0 -> (none); limit lower=-0.1 upper=0.1 effort=0 velocity=1.0 -> (none); type revolute -> fixed
- joint L4L3_J2: axis 0 0 1 -> (none); limit lower=-0.1 upper=0.1 effort=0 velocity=1.0 -> (none); type revolute -> fixed
- joint L5: axis 0 1 0 -> (none); limit lower=-0.1 upper=0.1 effort=0 velocity=1.0 -> (none); type revolute -> fixed
- joint L5L4_J1: axis 1 0 0 -> (none); limit lower=-0.1 upper=0.1 effort=0 velocity=1.0 -> (none); type revolute -> fixed
- joint L5L4_J2: axis 0 0 1 -> (none); limit lower=-0.1 upper=0.1 effort=0 velocity=1.0 -> (none); type revolute -> fixed
- joint SacrumL5_J1: axis 1 0 0 -> (none); limit lower=-0.1 upper=0.1 effort=0 velocity=1.0 -> (none); type revolute -> fixed
- joint SacrumL5_J2: axis 0 0 1 -> (none); limit lower=-0.1 upper=0.1 effort=0 velocity=1.0 -> (none); type revolute -> fixed
- joint Thorax: limit lower=-0.5 upper=0.6 effort=0 velocity=1.0 -> lower=-0.6 upper=0.7 effort=0 velocity=1.0

File: data/urdf/skeleton/skeleton_trunk.urdf (robot description, URDF)
Before this commit: robot skeleton_trunk, 31 links, 30 joints
Joints:
- joint L1: axis 0 1 0 -> (none); limit lower=-0.1 upper=0.1 effort=0 velocity=1.0 -> (none); type revolute -> fixed
- joint L1Thorax_J1: limit lower=-0.2 upper=0.2 effort=0 velocity=1.0 -> lower=-0.3 upper=0.3 effort=0 velocity=1.0
- joint L2: axis 0 1 0 -> (none); limit lower=-0.1 upper=0.1 effort=0 velocity=1.0 -> (none); type revolute -> fixed
- joint L2L1_J1: axis 1 0 0 -> (none); limit lower=-0.1 upper=0.1 effort=0 velocity=1.0 -> (none); type revolute -> fixed
- joint L2L1_J2: axis 0 0 1 -> (none); limit lower=-0.1 upper=0.1 effort=0 velocity=1.0 -> (none); type revolute -> fixed
- joint L3: axis 0 1 0 -> (none); limit lower=-0.1 upper=0.1 effort=0 velocity=1.0 -> (none); type revolute -> fixed
- joint L3L2_J1: axis 1 0 0 -> (none); limit lower=-0.1 upper=0.1 effort=0 velocity=1.0 -> (none); type revolute -> fixed
- joint L3L2_J2: axis 0 0 1 -> (none); limit lower=-0.1 upper=0.1 effort=0 velocity=1.0 -> (none); type revolute -> fixed
- joint L4: axis 0 1 0 -> (none); limit lower=-0.1 upper=0.1 effort=0 velocity=1.0 -> (none); type revolute -> fixed
- joint L4L3_J1: axis 1 0 0 -> (none); limit lower=-0.1 upper=0.1 effort=0 velocity=1.0 -> (none); type revolute -> fixed
- joint L4L3_J2: axis 0 0 1 -> (none); limit lower=-0.1 upper=0.1 effort=0 velocity=1.0 -> (none); type revolute -> fixed
- joint L5: axis 0 1 0 -> (none); limit lower=-0.1 upper=0.1 effort=0 velocity=1.0 -> (none); type revolute -> fixed
- joint L5L4_J1: axis 1 0 0 -> (none); limit lower=-0.1 upper=0.1 effort=0 velocity=1.0 -> (none); type revolute -> fixed
- joint L5L4_J2: axis 0 0 1 -> (none); limit lower=-0.1 upper=0.1 effort=0 velocity=1.0 -> (none); type revolute -> fixed
- joint SacrumL5_J1: axis 1 0 0 -> (none); limit lower=-0.1 upper=0.1 effort=0 velocity=1.0 -> (none); type revolute -> fixed
- joint SacrumL5_J2: axis 0 0 1 -> (none); limit lower=-0.1 upper=0.1 effort=0 velocity=1.0 -> (none); type revolute -> fixed
- joint Thorax: limit lower=-0.5 upper=0.6 effort=0 velocity=1.0 -> lower=-0.6 upper=0.7 effort=0 velocity=1.0

Commit message: Update skeleton urdf and scripts for COM projection

File: data/urdf/skeleton/LFootSphere.urdf (robot description, URDF)
Before this commit: robot LFootSphere, 28 links, 27 joints
Links:
- added link base_link_comshift
Joints:
- added joint base_link_comshift_J: type fixed, parent base_link_comshift, child Pelvis, origin xyz=-0.1 0 -0.04 rpy=0 0 0
- joint base_link_J: child Pelvis -> base_link_comshift

File: data/urdf/skeleton/LHandSphere.urdf (robot description, URDF)
Before this commit: robot LHandSphere, 28 links, 27 joints
Links:
- added link base_link_comshift
Joints:
- added joint base_link_comshift_J: type fixed, parent base_link_comshift, child Pelvis, origin xyz=-0.1 0 -0.04 rpy=0 0 0
- joint base_link_J: child Pelvis -> base_link_comshift

File: data/urdf/skeleton/RFootSphere.urdf (robot description, URDF)
Before this commit: robot RFootSphere, 28 links, 27 joints
Links:
- added link base_link_comshift
Joints:
- added joint base_link_comshift_J: type fixed, parent base_link_comshift, child Pelvis, origin xyz=-0.1 0 -0.04 rpy=0 0 0
- joint base_link_J: child Pelvis -> base_link_comshift

File: data/urdf/skeleton/RHandSphere.urdf (robot description, URDF)
Before this commit: robot RHandSphere, 28 links, 27 joints
Links:
- added link base_link_comshift
Joints:
- added joint base_link_comshift_J: type fixed, parent base_link_comshift, child Pelvis, origin xyz=-0.1 0 -0.04 rpy=0 0 0
- joint base_link_J: child Pelvis -> base_link_comshift

File: data/urdf/skeleton/skeleton.urdf (robot description, URDF)
Before this commit: robot skeleton, 58 links, 57 joints
Links:
- added link base_link_comshift
- added link base_link_visual; visual sphere radius=0.02
Joints:
- added joint base_link_comshift_J: type fixed, parent base_link_comshift, child Pelvis, origin xyz=-0.1 0 -0.04 rpy=0 0 0
- added joint base_link_visual_J: type fixed, parent base_link, child base_link_visual, origin xyz=0 0 0 rpy=0 0 0
- joint base_link_J: child Pelvis -> base_link_comshift

File: data/urdf/skeleton/skeleton_trunk.urdf (robot description, URDF)
Before this commit: robot skeleton_trunk, 31 links, 30 joints
Links:
- added link base_link_comshift
Joints:
- added joint base_link_comshift_J: type fixed, parent base_link_comshift, child Pelvis, origin xyz=-0.1 0 -0.04 rpy=0 0 0
- joint base_link_J: child Pelvis -> base_link_comshift
