Commit message: Add functions and fix Skeleton URDF:
* Add functions to get the list of takeoff and landing velocities of each waypoints of a path.
* Fix Skeleton URDF: rename some joints to order the trunk and full kinematic chains the same way.

File: data/urdf/skeleton/skeleton.urdf (robot description, URDF)
Before this commit: robot skeleton, 60 links, 59 joints
Joints:
- removed joint PelvisSacrum_J1
- removed joint ThoraxSkull_J1
- added joint A_PelvisSacrum_J1: type revolute, parent Pelvis, child PelvisSacrum_J1, origin xyz=-0.010389 0 0.018889 rpy=0 0 0, axis 1 0 0, limit lower=-0.2 upper=0.2 effort=0 velocity=1.0
- added joint A_ThoraxSkull_J1: type revolute, parent Thorax, child ThoraxSkull_J1, origin xyz=0.0037778 0 0.42122 rpy=0 0 0, axis 1 0 0, limit lower=-0.3 upper=0.3 effort=0 velocity=1.0

File: data/urdf/skeleton/skeleton_trunk_flexible.urdf (robot description, URDF)
Before this commit: robot skeleton_trunk_flexible, 26 links, 25 joints
Joints:
- removed joint PelvisSacrum_J1
- removed joint ThoraxSkull_J1
- added joint A_PelvisSacrum_J1: type revolute, parent Pelvis, child PelvisSacrum_J1, origin xyz=-0.010389 0 0.018889 rpy=0 0 0, axis 1 0 0, limit lower=-0.2 upper=0.2 effort=0 velocity=1.0
- added joint A_ThoraxSkull_J1: type revolute, parent Thorax, child ThoraxSkull_J1, origin xyz=0.0037778 0 0.42122 rpy=0 0 0, axis 1 0 0, limit lower=-0.3 upper=0.3 effort=0 velocity=1.0

Commit message: Fix URDF: remove collision for effector-spheres, increase size of spiderman trunk boxes

File: data/urdf/skeleton/skeleton.urdf (robot description, URDF)
Before this commit: robot skeleton, 60 links, 59 joints
Links:
- link LFootSphere: geometry visual sphere radius=0.01
- link LHandSphere: geometry visual sphere radius=0.01
- link RFootSphere: geometry visual sphere radius=0.01
- link RHandSphere: geometry visual sphere radius=0.01

File: data/urdf/spiderman/spiderman.urdf (robot description, URDF)
Before this commit: robot spiderman, 38 links, 37 joints
Links:
- link SpidermanLFootSphere: geometry visual sphere radius=0.01
- link SpidermanLHandSphere: geometry visual sphere radius=0.01
- link SpidermanRFootSphere: geometry visual sphere radius=0.01
- link SpidermanRHandSphere: geometry visual sphere radius=0.01
Joints:
- joint SpidermanLFootSphere: origin xyz=0.00134 -0.16 -0.09568 rpy=0 0 0 -> xyz=0.00134 -0.1 -0.09568 rpy=0 0 0
- joint SpidermanLHandSphere: origin xyz=-0.003 -0.0434 -0.0727 rpy=0 0.2 3.3415 -> xyz=0 -0.0434 -0.08 rpy=0 0.2 3.3415
- joint SpidermanRFootSphere: origin xyz=-0.00134 -0.16 -0.09568 rpy=0 0 0 -> xyz=-0.00134 -0.1 -0.09568 rpy=0 0 0
- joint SpidermanRHandSphere: origin xyz=0.0034 -0.0434 -0.0752 rpy=0 0.2 -0.2 -> xyz=0 -0.0434 -0.08 rpy=0 0.2 -0.2

Commit message: separate amrlessSkeleton scripts, flexion pose for full-skeleton

File: data/urdf/skeleton/skeleton.urdf (robot description, URDF)
Before this commit: robot skeleton, 60 links, 59 joints
Joints:
- joint LAnkle_J1: limit lower=-1.2 upper=1.2 effort=0 velocity=1.0 -> lower=-1.4 upper=1.2 effort=0 velocity=1.0
- joint LShank: limit lower=-0.05 upper=2.3 effort=0 velocity=1.0 -> lower=-0.05 upper=2.4 effort=0 velocity=1.0
- joint RAnkle_J1: limit lower=-1.2 upper=1.2 effort=0 velocity=1.0 -> lower=-1.4 upper=1.2 effort=0 velocity=1.0
- joint RShank: limit lower=-0.05 upper=2.3 effort=0 velocity=1.0 -> lower=-0.05 upper=2.4 effort=0 velocity=1.0

Commit message: Add toe DOF to skeleton, update key-configs

File: data/urdf/skeleton/skeleton.urdf (robot description, URDF)
Before this commit: robot skeleton, 60 links, 59 joints
Links:
- removed link LFootInter
- removed link LForearm_Virtual
- removed link RFootInter
- removed link RForearm_Virtual
- added link LFootToe, mass 0.2; collision mesh filename=package://hpp-rbprm-corba/meshes/skeleton/LFootToe.stl; visual mesh filename=package://hpp-rbprm-corba/meshes/skeleton/LFootToe.stl
- added link RFootToe, mass 0.2; collision mesh filename=package://hpp-rbprm-corba/meshes/skeleton/RFootToe.stl; visual mesh filename=package://hpp-rbprm-corba/meshes/skeleton/RFootToe.stl
Joints:
- removed joint LFootInter
- removed joint LForearm_Virtual
- removed joint RFootInter
- removed joint RForearm_Virtual
- added joint LFootToe: type revolute, parent LFoot, child LFootToe, origin xyz=0.1114 0.0168 -0.0571 rpy=0 0 0, axis 0 1 0, limit lower=-0.5 upper=0.5 effort=0 velocity=1.0
- added joint RFootToe: type revolute, parent RFoot, child RFootToe, origin xyz=0.1162 -0.0175 -0.0583 rpy=0 0 0, axis 0 1 0, limit lower=-0.5 upper=0.5 effort=0 velocity=1.0
- joint LFoot: child LFootInter -> LFoot
- joint LFootSphere: origin xyz=0.15 0.023 -0.095 rpy=0 0 0 -> xyz=0.0195 0.0044 -0.0159 rpy=0 0 0; parent LFoot -> LFootToe
- joint RFoot: child RFootInter -> RFoot
- joint RFootSphere: origin xyz=0.15 -0.023 -0.095 rpy=0 0 0 -> xyz=0.0147 0 -0.0147 rpy=0 0 0; parent RFoot -> RFootToe

Commit message: Add function to compute contactCones from given configuration, and Skeleton ref configs:
-fix convex-cone intersection plots (origin of lines),
-fix Affordance or configValidation in Skeleton scripts,
-Skeleton ref configs are the ballistic-interpolation keyframes (2 different when making
of leaving contacts) -> UPDATE SKELETON SCRIPTS WITH THEM,
-adapt Skeleton joint bounds to new refs configs

File: data/urdf/skeleton/skeleton.urdf (robot description, URDF)
Before this commit: robot skeleton, 58 links, 57 joints
Joints:
- joint LHumerus: limit lower=-2.8 upper=0.5 effort=0 velocity=1.0 -> lower=-2.8 upper=1.7 effort=0 velocity=1.0
- joint LShank: limit lower=-0.05 upper=2.4 effort=0 velocity=1.0 -> lower=-0.05 upper=2.7 effort=0 velocity=1.0
- joint RHumerus: limit lower=-2.7 upper=0.5 effort=0 velocity=1.0 -> lower=-2.7 upper=1.7 effort=0 velocity=1.0
- joint RShank: limit lower=-0.05 upper=2.4 effort=0 velocity=1.0 -> lower=-0.05 upper=2.7 effort=0 velocity=1.0

Commit message: Add finalFlexionPose, update skeleton

File: data/urdf/skeleton/skeleton.urdf (robot description, URDF)
Before this commit: robot skeleton, 60 links, 59 joints
Joints:
- joint Sacrum: limit lower=-0.1 upper=0.3 effort=0 velocity=1.0 -> lower=-0.1 upper=0.5 effort=0 velocity=1.0
- joint Skull: limit lower=-1.1 upper=0.4 effort=0 velocity=1.0 -> lower=-1.1 upper=0.5 effort=0 velocity=1.0
