Commit message: Modifs (including masses) for Kangaroo

File: data/urdf/kangaroo/kangaroo.urdf (robot description, URDF)
Before this commit: robot kangaroo, 57 links, 56 joints
Links:
- link Head: mass 0 -> 5
- link LArm: mass 1 -> 1.4
- link LForearm: mass 1 -> 0.6
- link LHand: mass 1 -> 0.5
- link LShank: mass 1 -> 3
- link LThigh: mass 1 -> 7
- link Pelvis: mass 1 -> 19
- link RArm: mass 1 -> 1.4
- link RForearm: mass 1 -> 0.6
- link RHand: mass 1 -> 0.5
- link RShank: mass 1 -> 3
- link RThigh: mass 1 -> 7
- link Tail: mass 0 -> 5
- link Tailbase: mass 0 -> 6
- link Torso: mass 1 -> 25
